File: PCB/Console.kicad_pcb (KiCad board)
At the start: 2 copper layers, 168 x 72.5 mm, 171 parts, among them J1 Programming Header, J2 UART, J3 USB_B, J4 USB_A, J5 USB_A, J6 USB_A, J7 USB_A, J8 Barrel_Jack_Switch, J9 Programming Header, Q1 FDN338P, Q2 MMBT3904, Q3 FDN338P, SW1 SW_Push_LED, SW10 Rotary_Encoder_Switch, SW11 SW_Push, SW12 SW_Push, SW2 SW_Push_LED, SW3 SW_Push_LED, SW4 SW_Push_LED, SW5 SW_Push_LED, SW6 SW_Push_LED, SW7 Rotary_Encoder_Switch, SW8 Rotary_Encoder_Switch, SW9 Rotary_Encoder_Switch, U1 ATmega328P-PU, U10 NHD-3.12-25664UCW2, U2 MCP23017_SO, U3 CY7C65632-28LTXC, U5 MIC2027-2BM, U6 CP2102N-A02-GQFN20, U7 DMP1005UFDF, U8 AP2114HA-3.3TRG1, U9 ESP32-WROOM-32, Y1 16MHz, Y2 12MHz

Commit message: PCB "Complete", still needs checking etc
Parts:
- moved D9 23.5 mm to (185.0, 87.5), turned to 180 degrees
- moved R65 6.11 mm to (187.0, 81.0)
- moved R64 6.10 mm to (186.0, 81.0)
- moved R67 6.06 mm to (189.0, 81.0), turned to 270 degrees
- moved R66 4.25 mm to (188.0, 81.0), turned to 270 degrees
- moved U5 3.86 mm to (196.0, 83.5)
- moved C24 3.58 mm to (158.2, 99.0)
- moved C19 1.10 mm to (182.6, 89.5)
- moved U3 0.20 mm to (180.6, 84.0)
- moved Y2 0.20 mm to (180.2, 89.5)
Routing:
- net /USB Hub and Serial Converter/VBUS_B: track 5.07 -> 59.1 mm
- net +3V3: track 555.0 -> 599.4 mm, vias 24 -> 31
- net /USB Hub and Serial Converter/D1P: track 0.00 -> 43.6 mm, vias 0 -> 2
- net /USB Hub and Serial Converter/D1N: track 0.00 -> 43.3 mm, vias 0 -> 2
- net /USB Hub and Serial Converter/VBUS_A: track 0.00 -> 33.3 mm, vias 0 -> 1
- net /USB Hub and Serial Converter/D4N: track 0.00 -> 32.8 mm, vias 0 -> 1
- net /USB Hub and Serial Converter/D4P: track 0.00 -> 31.5 mm, vias 0 -> 1
- net Net-(C27-Pad2): track 0.00 -> 31.2 mm
- net /USB Hub and Serial Converter/D3N: track 0.00 -> 24.9 mm, vias 0 -> 1
- net /USB Hub and Serial Converter/D3P: track 0.00 -> 24.2 mm, vias 0 -> 1
- net /USB Hub and Serial Converter/DIN_P: track 0.00 -> 23.8 mm, vias 0 -> 2
- net Net-(C33-Pad2): track 0.00 -> 23.8 mm
- net /USB Hub and Serial Converter/DIN_N: track 0.00 -> 22.9 mm, vias 0 -> 2
- net /USB Hub and Serial Converter/~OVR4: track 0.00 -> 21.1 mm, vias 0 -> 2
- net /USB Hub and Serial Converter/~OVR3: track 0.00 -> 21.0 mm, vias 0 -> 2
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
Commit message: PCB Version 1: As Sent to Fab
Parts:
- added C20: 0.1uF, Capacitor_SMD:C_0603_1608Metric, F.Cu at (195.5, 76.5)
- added C23: 0.1uF, Capacitor_SMD:C_0603_1608Metric, F.Cu at (196.5, 78.5)
- added D17: LED, LED_SMD:LED_0603_1608Metric, F.Cu at (164.8, 129.2)
- added H10: MountingHole, Symbol:OSHW-Logo_5.7x6mm_SilkScreen, F.Cu at (149.5, 116.5)
- added H11: MountingHole, Symbol:KiCad-Logo2_5mm_SilkScreen, F.Cu at (218.2, 62.3)
- added R12: 10k, Resistor_SMD:R_0402_1005Metric, F.Cu at (188.0, 78.7)
- added R13: 10k, Resistor_SMD:R_0402_1005Metric, F.Cu at (189.0, 78.8)
- added R14: DNP, Resistor_SMD:R_0402_1005Metric, F.Cu at (190.2, 78.7)
- added R32: 10K, Resistor_SMD:R_0402_1005Metric, F.Cu at (191.8, 78.2)
- added R33: 270R, Resistor_SMD:R_0402_1005Metric, F.Cu at (162.0, 129.2)
- added R68: 10k, Resistor_SMD:R_0402_1005Metric, F.Cu at (137.5, 102.0)
- added R69: 10k, Resistor_SMD:R_0402_1005Metric, F.Cu at (136.2, 102.0)
- added TP2: TestPoint, TestPoint:TestPoint_Pad_1.5x1.5mm, F.Cu at (189.5, 68.8)
- added TP3: TestPoint, TestPoint:TestPoint_Pad_1.5x1.5mm, F.Cu at (192.2, 68.8)
- added U4: 24LC02, Package_SO:SOIC-8_3.9x4.9mm_P1.27mm, F.Cu at (191.0, 74.0)
- moved D1 30.1 mm to (73.5, 129.3)
- moved R1 29.3 mm to (75.8, 128.8), turned to 270 degrees
- moved C4 1.17 mm to (97.6, 107.5)
- moved R5 0.58 mm to (219.8, 107.0)
- moved R3 0.54 mm to (181.7, 107.0)
- moved R4 0.52 mm to (200.7, 107.0)
- moved H3 0.50 mm to (190.5, 62.0)
- moved SW12 0.45 mm to (146.3, 128.0)
- moved C25 0.35 mm to (215.6, 87.2)
- moved R8 0.30 mm to (219.8, 125.5)
- moved C30 0.25 mm to (209.8, 88.5)
- moved J2 0.25 mm to (97.0, 100.8)
- moved R20 0.25 mm to (140.8, 103.3)
- moved R6 0.20 mm to (181.7, 125.5)
- moved R7 0.20 mm to (200.7, 125.5)
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Connections:
- U7 pad 8: (no net) -> /Power/VCC_IN
- U9 pad 30: Net-(U9-Pad30) -> /Core/LED
Routing:
- net /Core/LED: track 0.00 -> 44.6 mm, vias 0 -> 2
- net /Peripherals/LED: track 2.49 -> 39.7 mm, vias 0 -> 2
- net /USB Hub and Serial Converter/EEPROM_SCL: track 0.00 -> 30.0 mm, vias 0 -> 3
- net /USB Hub and Serial Converter/EEPROM_SDA: track 0.00 -> 29.4 mm, vias 0 -> 3
- net +3V3: track 599.4 -> 614.4 mm, vias 31 -> 32
- net /USB Hub and Serial Converter/DIN_N: track 22.9 -> 13.0 mm, vias 2 -> 1
- net /USB Hub and Serial Converter/DIN_P: track 23.8 -> 14.6 mm, vias 2 -> 1
- net /Core/SDA: track 66.4 -> 72.5 mm
- net +5V: track 103.3 -> 108.8 mm
- net /Peripherals/SW_5: track 28.0 -> 32.7 mm
- net /Peripherals/SW_6: track 48.4 -> 51.6 mm
- net /Peripherals/SW_3: track 53.1 -> 56.1 mm
- net Net-(R14-Pad2): track 0.00 -> 2.94 mm
- net Net-(C27-Pad2): track 31.2 -> 33.6 mm
- net VBUS: track 55.3 -> 57.1 mm, vias 4 -> 6
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Other:
- board text added: "ekafarowski.com"
- board text added: "github.com/Aliasmk/EMRSNxEOS"
- board text added: "michael.kafarowski.com"
