File: PCB/Console.sch (KiCad schematic (older format))
At the start: 0 parts

Commit message: Schematic, Code Refactor, 328P workspace
Parts:
- added C1: 0.1uF, symbol Device:C
- added C2, C3: 4.7uF, symbol Device:C
- added J1: Barrel_Jack_Switch, symbol Connector:Barrel_Jack_Switch
- added U1: AP2114HA-3.3TRG1, TO_SOT_Packages_SMD:SOT-223-3_TabPin2, symbol MK_Library:AP2114-HA
Connections:
- new net +3V3: C3.1, U1.3 (VOUT)
- new net +5V: C1.1, C2.1, J1.1, U1.1 (VIN)
- new net GND: C1.2, C2.2, C3.2, J1.2, U1.2 (GND)
- no-connect marks 0 -> 2
Other:
- note added: "Power Input:\n5V, 1.5A DC"

Commit message: WIP PCB changes
Parts:
- removed C1: 0.1uF, symbol Device:C
- removed C2, C3: 4.7uF, symbol Device:C
- removed J1: Barrel_Jack_Switch, symbol Connector:Barrel_Jack_Switch
- removed U1: AP2114HA-3.3TRG1, TO_SOT_Packages_SMD:SOT-223-3_TabPin2, symbol MK_Library:AP2114-HA
- added H1, H2, H3, H4, H5, H6, H7, H8: MountingHole, MountingHole:MountingHole_2.7mm_M2.5, symbol Mechanical:MountingHole
- added H9: MountingHole, EMRSNxEOS:Ghost, symbol Mechanical:MountingHole
Connections:
- no-connect marks 2 -> 0
Other:
- note removed: "Power Input:\n5V, 1.5A DC"

Commit message: PCB Version 1: As Sent to Fab
Parts:
- added H10: MountingHole, Symbol:OSHW-Logo_5.7x6mm_SilkScreen, symbol Mechanical:MountingHole
- added H11: MountingHole, Symbol:KiCad-Logo2_5mm_SilkScreen, symbol Mechanical:MountingHole
Changed lines of the file:
@@
+	1    0    0    -1
+$EndComp
+$Comp
+L Graphic:Logo_Open_Hardware_Small #LOGO1
+U 1 1 5FB483D2
+P 800 7700
+F 0 "#LOGO1" H 800 7975 50  0001 C CNN
+F 1 "Logo_Open_Hardware_Small" H 800 7475 50  0001 C CNN
+F 2 "" H 800 7700 50  0001 C CNN
+F 3 "~" H 800 7700 50  0001 C CNN
+	1    800  7700
+	1    0    0    -1
+$EndComp
+$Comp
+L Mechanical:MountingHole H10
+U 1 1 5FB48A85
+P 5800 7500
+F 0 "H10" H 5900 7546 50  0000 L CNN
+F 1 "MountingHole" H 5900 7455 50  0000 L CNN
+F 2 "Symbol:OSHW-Logo_5.7x6mm_SilkScreen" H 5800 7500 50  0001 C CNN
+F 3 "~" H 5800 7500 50  0001 C CNN
+	1    5800 7500
+	1    0    0    -1
+$EndComp
+$Comp
+L Mechanical:MountingHole H11
+U 1 1 5FB1B00A
+P 5800 7250
+F 0 "H11" H 5900 7296 50  0000 L CNN
+F 1 "MountingHole" H 5900 7205 50  0000 L CNN
+F 2 "Symbol:KiCad-Logo2_5mm_SilkScreen" H 5800 7250 50  0001 C CNN
+F 3 "~" H 5800 7250 50  0001 C CNN
+	1    5800 7250
 	1    0    0    -1
 $EndComp
