File: PCB/Core.sch (KiCad schematic (older format))
At the start: 1 part

Commit message: Schematic, Code Refactor, 328P workspace
Parts:
- added C4: 22uF, symbol Device:C_Small
- added C40, C5: 0.1uF, symbol Device:C_Small
- added C6: C_Small, symbol Device:C_Small
- added J2: Programming Header, symbol Connector_Generic:Conn_01x04
- added JP1: BS1_Sel, symbol Jumper:SolderJumper_2_Open
- added JP2: BS2_Sel, symbol Jumper:SolderJumper_2_Open
- added R1, R2, R3: 10k, symbol Device:R
- added SW1, SW12: SW_Push, symbol Switch:SW_Push
- added U3: NHD-3.12-25664UCW2, symbol MK_Library:NHD-3.12-25664UCW2
- gave numbers to parts that had none: 1
Connections:
- net GND: now reaches U2.1 (GND), U2.15 (GND), U2.38 (GND), U2.39 (GND)
- net GND: now also C4.2, C40.1, C5.2, C6.2, J2.4 (Pin_4), R2.2, R3.2, SW1.2, SW12.1, U3.1 (VSS), U3.17 (~CS)
- net SUSPEND_SENSE: now reaches U2.10 (IO25)
- net BTN_INT: now reaches U2.11 (IO26)
- net OLED_D1: now reaches U2.13 (IO14)
- net OLED_D1: now also U3.8 (DB1/SDIN)
- net OLED_EN: now reaches U2.14 (IO12)
- net OLED_EN: now also U3.6 (EN)
- net OLED_D0: now reaches U2.16 (IO13)
- net OLED_D0: now also U3.7 (DB0/SCLK)
- net +3V3: now reaches U2.2 (VDD)
- net +3V3: now also C4.1, C6.1, J2.1 (Pin_1), JP1.1 (A), JP2.1 (A), R1.1, U3.16 (~RESET), U3.2 (VDD)
- net OLED_D2: now reaches U2.23 (IO15)
- net OLED_D2: now also U3.9 (DB2/NC)
- net LED_PWM: now reaches U2.24 (IO2)
- net BOOT: now reaches U2.25 (IO0)
- net BOOT: now also C40.2, SW1.1
- net OLED_DC: now reaches U2.26 (IO4)
- net OLED_DC: now also U3.4 (D/C)
- net OLED_D3: now reaches U2.27 (IO16)
- net OLED_D3: now also U3.10 (DB3/VSS)
- net OLED_D4: now reaches U2.28 (IO17)
- net OLED_D4: now also U3.11 (DB4/VSS)
- net OLED_RW: now reaches U2.29 (IO5)
- net OLED_RW: now also U3.5 (R/W)
- net EN: now reaches U2.3 (EN)
- net EN: now also C5.1, R1.2, SW12.2
- net OLED_D5: now reaches U2.30 (IO18)
- net OLED_D5: now also U3.12 (DB5/VSS)
- net OLED_D6: now reaches U2.31 (IO19)
- net OLED_D6: now also U3.13 (DB6/VSS)
- net OLED_D7: now reaches U2.33 (IO21)
- net OLED_D7: now also U3.14 (DB7/VSS)
- net RXD0: now reaches U2.34 (RXD0/IO3)
- net RXD0: now also J2.3 (Pin_3)
- net TXD0: now reaches U2.35 (TXD0/IO1)
- net TXD0: now also J2.2 (Pin_2)
- net SDA: now reaches U2.36 (IO22)
- net SCL: now reaches U2.37 (IO23)
- new net: JP1.2 (B), R2.1, U3.19 (BS1)
- new net: JP2.2 (B), R3.1, U3.20 (BS2)
- no-connect marks 0 -> 13
Other:
- note added: "ESP32 Main Processor"
- note added: "OLED Display"
- moved on the sheet: U2

Commit message: WIP PCB changes
Parts:
- removed JP1: BS1_Sel, symbol Jumper:SolderJumper_2_Open
- removed JP2: BS2_Sel, symbol Jumper:SolderJumper_2_Open
- removed R2, R3: 10k, symbol Device:R
- C39: renamed from C4; footprint (none) -> Capacitor_SMD:C_0805_2012Metric; Digikey (none) -> 1276-6687-1-ND; MPN (none) -> CL21A226KQCLRNC; Manufacturer (none) -> Samsung
- C40: renamed from C5; footprint (none) -> Capacitor_SMD:C_0603_1608Metric; Digikey (none) -> 311-4046-1-ND; MPN (none) -> CC0603KRX5R9BB104; Manufacturer (none) -> Yageo
- C41: renamed from C40; footprint (none) -> Capacitor_SMD:C_0603_1608Metric; Digikey (none) -> 311-4046-1-ND; MPN (none) -> CC0603KRX5R9BB104; Manufacturer (none) -> Yageo
- C42: renamed from C6; value C_Small -> 1uF; footprint (none) -> Capacitor_SMD:C_0603_1608Metric; Digikey (none) -> 1276-1102-1-ND; MPN (none) -> CL10A105KA8NNNC; Manufacturer (none) -> Samsung
- J9: renamed from J2; footprint (none) -> Connector_PinSocket_1.27mm:PinSocket_1x04_P1.27mm_Vertical; Digikey (none) -> 2057-PH1-04-UA-ND; MPN (none) -> PH1-04-UA; Manufacturer (none) -> Adam Tech
- R31: renamed from R1; footprint (none) -> Resistor_SMD:R_0402_1005Metric; Digikey (none) -> RMCF0402FT10K0CT-ND; MPN (none) -> RMCF0402FT10K0; Manufacturer (none) -> Stackpole
- SW11: renamed from SW12; footprint (none) -> MK_Library:PTS636 SK25F SMTR LFS; Digikey (none) -> CKN12330-1-ND; MPN (none) -> PTS636 SK25F SMTR LFS; Manufacturer (none) -> C&K
- SW12: renamed from SW1; footprint (none) -> MK_Library:PTS636 SK25F SMTR LFS; Digikey (none) -> CKN12330-1-ND; MPN (none) -> PTS636 SK25F SMTR LFS; Manufacturer (none) -> C&K
- U10: renamed from U3; footprint (none) -> Connector_PinSocket_2.54mm:PinSocket_1x20_P2.54mm_Vertical; Digikey (none) -> NHD-3.12-25664UCW2-ND; MPN (none) -> NHD-3.12-25664UCW2; Manufacturer (none) -> Newhaven Display Intl
- U9: renamed from U2; Digikey (none) -> 1904-1028-1-ND; MPN (none) -> ESP32-WROOM-32U (16MB); Manufacturer (none) -> Espressif Systems
Connections:
- net +3V3: no longer U10.16 (~RESET)
- net BTN_INT: now also U9.31 (IO19); no longer U9.11 (IO26)
- net GND: no longer U10.17 (~CS)
- net LED_PWM: now also U9.29 (IO5); no longer U9.24 (IO2)
- net OLED_D0: now also U9.9 (IO33); no longer U9.16 (IO13)
- net OLED_D1: now also U9.10 (IO25); no longer U9.13 (IO14)
- net OLED_D2: now also U9.11 (IO26); no longer U9.23 (IO15)
- net OLED_D3: now also U9.12 (IO27); no longer U9.27 (IO16)
- net OLED_D4: now also U9.13 (IO14); no longer U9.28 (IO17)
- net OLED_D5: now also U9.14 (IO12); no longer U9.30 (IO18)
- net OLED_D6: now also U9.16 (IO13); no longer U9.31 (IO19)
- net OLED_D7: now also U9.23 (IO15); no longer U9.33 (IO21)
- net OLED_DC: now also U9.6 (IO34); no longer U9.26 (IO4)
- net OLED_EN: now also U9.8 (IO32); no longer U9.14 (IO12)
- net OLED_RW: now also U9.7 (IO35); no longer U9.29 (IO5)
- net SUSPEND_SENSE: now also U9.33 (IO21); no longer U9.10 (IO25)
- net OLED_BS1: now reaches U10.19 (BS1)
- net OLED_BS1: now also U9.27 (IO16)
- net OLED_BS2: now reaches U10.20 (BS2)
- net OLED_BS2: now also U9.28 (IO17)
- new net OLED_~CS: U10.17 (~CS), U9.26 (IO4)
- new net OLED_~RESET: U10.16 (~RESET), U9.24 (IO2)
- no-connect marks 13 -> 8

Commit message: PCB Version 1: As Sent to Fab
Parts:
- added D17: LED_Green, LED_SMD:LED_0603_1608Metric, symbol Device:LED
- added R33: 270R, Resistor_SMD:R_0402_1005Metric, symbol Device:R
- added R68, R69: 10k, Resistor_SMD:R_0402_1005Metric, symbol Device:R
- C40, C41: Digikey 311-4046-1-ND -> 587-1243-1-ND; MPN CC0603KRX5R9BB104 -> UMK107B7104KA-T; Manufacturer Yageo -> Taiyo Yuden
Connections:
- net +3V3: now also R68.1, R69.1
- net GND: now also D17.1 (K)
- net SCL: now also R69.2
- net SDA: now also R68.2
- net LED: now reaches U9.30 (IO18)
- net LED: now also R33.1
- new net: D17.2 (A), R33.2
Other:
- moved on the sheet: J9
Changed lines of the file:
@@
 	10250 3050 10050 3050
 Wire Wire Line
-	5800 4000 6400 4000
-Wire Wire Line
-	5800 4100 6400 4100
-Text Label 6400 4000 2    50   ~ 0
+	5800 4000 6700 4000
+Wire Wire Line
+	5800 4100 7000 4100
+Text Label 7300 4000 2    50   ~ 0
 SDA
-Text Label 6400 4100 2    50   ~ 0
+Text Label 7300 4100 2    50   ~ 0
 SCL
 Wire Wire Line
@@
 L Connector_Generic:Conn_01x04 J9
 U 1 1 5FC9AD65
-P 3850 5450
-F 0 "J9" H 3768 5767 50  0000 C CNN
-F 1 "Programming Header" H 3768 5676 50  0000 C CNN
-F 2 "Connector_PinSocket_1.27mm:PinSocket_1x04_P1.27mm_Vertical" H 3850 5450 50  0001 C CNN
-F 3 "~" H 3850 5450 50  0001 C CNN
-F 4 "2057-PH1-04-UA-ND" H 3850 5450 50  0001 C CNN "Digikey"
-F 5 "PH1-04-UA" H 3850 5450 50  0001 C CNN "MPN"
-F 6 "Adam Tech" H 3850 5450 50  0001 C CNN "Manufacturer"
-	1    3850 5450
+P 3550 5600
+F 0 "J9" H 3468 5917 50  0000 C CNN
+F 1 "Programming Header" H 3468 5826 50  0000 C CNN
+F 2 "Connector_PinSocket_1.27mm:PinSocket_1x04_P1.27mm_Vertical" H 3550 5600 50  0001 C CNN
+F 3 "~" H 3550 5600 50  0001 C CNN
+F 4 "2057-PH1-04-UA-ND" H 3550 5600 50  0001 C CNN "Digikey"
+F 5 "PH1-04-UA" H 3550 5600 50  0001 C CNN "MPN"
+F 6 "Adam Tech" H 3550 5600 50  0001 C CNN "Manufacturer"
+	1    3550 5600
 	-1   0    0    -1
 $EndComp
 Wire Wire Line
-	4050 5350 4600 5350
+	3750 5500 4300 5500
 $Comp
 L power:+3V3 #PWR0124
 U 1 1 5FC9DB9C
-P 4600 5300
-F 0 "#PWR0124" H 4600 5150 50  0001 C CNN
-F 1 "+3V3" H 4615 5473 50  0000 C CNN
-F 2 "" H 4600 5300 50  0001 C CNN
-F 3 "" H 4600 5300 50  0001 C CNN
-	1    4600 5300
+P 4300 5450
+F 0 "#PWR0124" H 4300 5300 50  0001 C CNN
+F 1 "+3V3" H 4315 5623 50  0000 C CNN
+F 2 "" H 4300 5450 50  0001 C CNN
+F 3 "" H 4300 5450 50  0001 C CNN
+	1    4300 5450
 	1    0    0    -1
 $EndComp
 Wire Wire Line
-	4600 5300 4600 5350
-Wire Wire Line
-	4050 5650 4600 5650
-Wire Wire Line
-	4600 5650 4600 5700
+	4300 5450 4300 5500
+Wire Wire Line
+	3750 5800 4300 5800
+Wire Wire Line
+	4300 5800 4300 5850
 $Comp
 L power:GND #PWR0125
 U 1 1 5FCA2179
-P 4600 5700
-F 0 "#PWR0125" H 4600 5450 50  0001 C CNN
-F 1 "GND" H 4605 5527 50  0000 C CNN
-F 2 "" H 4600 5700 50  0001 C CNN
-F 3 "" H 4600 5700 50  0001 C CNN
-	1    4600 5700
+P 4300 5850
+F 0 "#PWR0125" H 4300 5600 50  0001 C CNN
+F 1 "GND" H 4305 5677 50  0000 C CNN
+F 2 "" H 4300 5850 50  0001 C CNN
+F 3 "" H 4300 5850 50  0001 C CNN
+	1    4300 5850
 	1    0    0    -1
 $EndComp
 Wire Wire Line
-	4050 5450 4600 5450
-Wire Wire Line
-	4050 5550 4600 5550
-Text Label 4600 5450 2    50   ~ 0
+	3750 5600 4300 5600
+Wire Wire Line
+	3750 5700 4300 5700
+Text Label 4300 5600 2    50   ~ 0
 TXD0
-Text Label 4600 5550 2    50   ~ 0
+Text Label 4300 5700 2    50   ~ 0
 RXD0
 Wire Wire Line
@@
 F 2 "Capacitor_SMD:C_0603_1608Metric" H 4300 2700 50  0001 C CNN
 F 3 "~" H 4300 2700 50  0001 C CNN
-F 4 "311-4046-1-ND" H 4300 2700 50  0001 C CNN "Digikey"
-F 5 "CC0603KRX5R9BB104" H 4300 2700 50  0001 C CNN "MPN"
-F 6 "Yageo" H 4300 2700 50  0001 C CNN "Manufacturer"
+F 4 "587-1243-1-ND" H 4300 2700 50  0001 C CNN "Digikey"
+F 5 "UMK107B7104KA-T" H 4300 2700 50  0001 C CNN "MPN"
+F 6 "Taiyo Yuden" H 4300 2700 50  0001 C CNN "Manufacturer"
 	1    4300 2700
 	1    0    0    -1
@@
 F 2 "Capacitor_SMD:C_0603_1608Metric" H 6750 2650 50  0001 C CNN
 F 3 "~" H 6750 2650 50  0001 C CNN
-F 4 "311-4046-1-ND" H 6750 2650 50  0001 C CNN "Digikey"
-F 5 "CC0603KRX5R9BB104" H 6750 2650 50  0001 C CNN "MPN"
-F 6 "Yageo" H 6750 2650 50  0001 C CNN "Manufacturer"
+F 4 "587-1243-1-ND" H 6750 2650 50  0001 C CNN "Digikey"
+F 5 "UMK107B7104KA-T" H 6750 2650 50  0001 C CNN "MPN"
+F 6 "Taiyo Yuden" H 6750 2650 50  0001 C CNN "Manufacturer"
 	1    6750 2650
 	0    1    1    0
@@
 Text Label 6400 2900 2    50   ~ 0
 OLED_~CS
+Wire Wire Line
+	5800 3700 6400 3700
+Text Label 6400 3700 2    50   ~ 0
+LED
+$Comp
+L Device:R R?
+U 1 1 5FB56CC1
+P 2850 5350
+AR Path="/5F4A9E86/5FB56CC1" Ref="R?"  Part="1"
+AR Path="/5F4A9D3D/5FB56CC1" Ref="R33"  Part="1"
+F 0 "R33" H 2920 5396 50  0000 L CNN
+F 1 "270R" H 2920 5305 50  0000 L CNN
+F 2 "Resistor_SMD:R_0402_1005Metric" V 2780 5350 50  0001 C CNN
+F 3 "~" H 2850 5350 50  0001 C CNN
+F 4 "311-270JRCT-ND" H 2850 5350 50  0001 C CNN "Digikey"
+F 5 "RC0402JR-07270RL" H 2850 5350 50  0001 C CNN "MPN"
+F 6 "Yageo" H 2850 5350 50  0001 C CNN "Manufacturer"
+	1    2850 5350
+	1    0    0    -1
+$EndComp
+Wire Wire Line
+	2850 5200 2850 5150
+Wire Wire Line
+	2850 5150 2450 5150
+Text Label 2450 5150 0    50   ~ 0
+LED
+$Comp
+L Device:LED D?
+U 1 1 5FB56CCD
+P 2850 5750
+AR Path="/5F4A9E86/5FB56CCD" Ref="D?"  Part="1"
+AR Path="/5F4A9D3D/5FB56CCD" Ref="D17"  Part="1"
+F 0 "D17" V 2889 5633 50  0000 R CNN
+F 1 "LED_Green" V 2798 5633 50  0000 R CNN
+F 2 "LED_SMD:LED_0603_1608Metric" H 2850 5750 50  0001 C CNN
+F 3 "~" H 2850 5750 50  0001 C CNN
+F 4 "160-1446-1-ND" H 2850 5750 50  0001 C CNN "Digikey"
+F 5 "LTST-C191KGKT" H 2850 5750 50  0001 C CNN "MPN"
+F 6 "Lite-On Inc." H 2850 5750 50  0001 C CNN "Manufacturer"
+	1    2850 5750
+	0    -1   -1   0
+$EndComp
+Wire Wire Line
+	2850 5500 2850 5600
+Wire Wire Line
+	2850 5900 2850 6000
+$Comp
+L power:GND #PWR?
+U 1 1 5FB56CD5
+P 2850 6000
+AR Path="/5F4A9E86/5FB56CD5" Ref="#PWR?"  Part="1"
+AR Path="/5F4A9D3D/5FB56CD5" Ref="#PWR0129"  Part="1"
+F 0 "#PWR0129" H 2850 5750 50  0001 C CNN
+F 1 "GND" H 2855 5827 50  0000 C CNN
+F 2 "" H 2850 6000 50  0001 C CNN
+F 3 "" H 2850 6000 50  0001 C CNN
+	1    2850 6000
+	1    0    0    -1
+$EndComp
+$Comp
+L Device:R R68
+U 1 1 5FB663F5
+P 6700 3700
+F 0 "R68" H 6770 3746 50  0000 L CNN
+F 1 "10k" H 6770 3655 50  0000 L CNN
+F 2 "Resistor_SMD:R_0402_1005Metric" V 6630 3700 50  0001 C CNN
+F 3 "~" H 6700 3700 50  0001 C CNN
+F 4 "RMCF0402FT10K0CT-ND" H 6700 3700 50  0001 C CNN "Digikey"
+F 5 "RMCF0402FT10K0" H 6700 3700 50  0001 C CNN "MPN"
+F 6 "Stackpole" H 6700 3700 50  0001 C CNN "Manufacturer"
+	1    6700 3700
+	1    0    0    -1
+$EndComp
+$Comp
+L Device:R R69
+U 1 1 5FB6686A
+P 7000 3700
+F 0 "R69" H 7070 3746 50  0000 L CNN
+F 1 "10k" H 7070 3655 50  0000 L CNN
+F 2 "Resistor_SMD:R_0402_1005Metric" V 6930 3700 50  0001 C CNN
+F 3 "~" H 7000 3700 50  0001 C CNN
+F 4 "RMCF0402FT10K0CT-ND" H 7000 3700 50  0001 C CNN "Digikey"
+F 5 "RMCF0402FT10K0" H 7000 3700 50  0001 C CNN "MPN"
+F 6 "Stackpole" H 7000 3700 50  0001 C CNN "Manufacturer"
+	1    7000 3700
+	1    0    0    -1
+$EndComp
+Wire Wire Line
+	6700 3850 6700 4000
+Connection ~ 6700 4000
+Wire Wire Line
+	6700 4000 7300 4000
+Wire Wire Line
+	7000 3850 7000 4100
+Connection ~ 7000 4100
+Wire Wire Line
+	7000 4100 7300 4100
+$Comp
+L power:+3V3 #PWR0130
+U 1 1 5FB6C0F9
+P 6700 3550
+F 0 "#PWR0130" H 6700 3400 50  0001 C CNN
+F 1 "+3V3" H 6715 3723 50  0000 C CNN
+F 2 "" H 6700 3550 50  0001 C CNN
+F 3 "" H 6700 3550 50  0001 C CNN
+	1    6700 3550
+	1    0    0    -1
+$EndComp
+$Comp
+L power:+3V3 #PWR0131
+U 1 1 5FB6C4A4
+P 7000 3550
+F 0 "#PWR0131" H 7000 3400 50  0001 C CNN
+F 1 "+3V3" H 7015 3723 50  0000 C CNN
+F 2 "" H 7000 3550 50  0001 C CNN
+F 3 "" H 7000 3550 50  0001 C CNN
+	1    7000 3550
+	1    0    0    -1
+$EndComp
 $EndSCHEMATC
