File: PCB/EncoderCircuit.sch (KiCad schematic (older format))
At the start: 10 parts, among them SW8 Rotary_Encoder_Switch

Commit message: WIP PCB changes
Parts:
- removed R18, R19: 10K, symbol Device:R
- removed R20, R21, R22: 10k, symbol Device:R
- removed R23: R, symbol Device:R
- added R40, R41, R42, R43, R44, R45: 10K, Resistor_SMD:R_0402_1005Metric, symbol Device:R
- C6: renamed from C12; footprint (none) -> Capacitor_SMD:C_0402_1005Metric; Digikey (none) -> 311-1677-1-ND; MPN (none) -> CC0402JRX7R8BB103; Manufacturer (none) -> Yageo
- C7: renamed from C13; footprint (none) -> Capacitor_SMD:C_0402_1005Metric; Digikey (none) -> 311-1677-1-ND; MPN (none) -> CC0402JRX7R8BB103; Manufacturer (none) -> Yageo
- C8: renamed from C14; footprint (none) -> Capacitor_SMD:C_0402_1005Metric; Digikey (none) -> 311-1677-1-ND; MPN (none) -> CC0402JRX7R8BB103; Manufacturer (none) -> Yageo
- SW7: renamed from SW8; footprint (none) -> EMRSNxEOS:PEC12RHeader; Digikey (none) -> PEC11R-4220F-S0012-ND; MPN (none) -> PEC11R-4220F-S0012; Manufacturer (none) -> Bourns Inc.
Connections:
- net +3V3: now also R42.2, R43.2, R45.1
- net ENC_A: now also R40.2
- net ENC_B: now also R41.2
- net ENC_SW: now also R44.2, R45.2
- net GND: now also SW7.C
- net at SW7.A: now also R40.1, R43.1
- net at SW7.B: now also R41.1, R42.1
- net at SW7.S1: now also R44.1
- no-connect marks 1 -> 0
Other:
- moved on the sheet: C6, C7, C8

Commit message: PCB Version 1: As Sent to Fab
Parts:
- R40, R41, R42, R43, R44, R45: value 10K -> 10k; Digikey (none) -> RMCF0402FT10K0CT-ND; MPN (none) -> RMCF0402FT10K0; Manufacturer (none) -> Stackpole
Changed lines of the file:
@@
 AR Path="/5F4A9E86/5F6DDF02/5F69EEA5" Ref="SW10"  Part="1"
 AR Path="/5F4A9E86/5F60074F/5F69EEA5" Ref="SW?"  Part="1"
-F 0 "SW7" H 5950 4050 50  0000 C CNN
+F 0 "SW10" H 5950 4050 50  0000 C CNN
 F 1 "Rotary_Encoder_Switch" H 5750 3550 50  0000 C CNN
 F 2 "EMRSNxEOS:PEC12RHeader" H 5800 3960 50  0001 C CNN
@@
 AR Path="/5F4A9E86/5F6DDF02/5F6A38A0" Ref="C17"  Part="1"
 AR Path="/5F4A9E86/5F60074F/5F6A38A0" Ref="C?"  Part="1"
-F 0 "C8" H 6865 3996 50  0000 L CNN
+F 0 "C17" H 6865 3996 50  0000 L CNN
 F 1 "10n" H 6865 3905 50  0000 L CNN
 F 2 "Capacitor_SMD:C_0402_1005Metric" H 6788 3800 50  0001 C CNN
@@
 AR Path="/5F4A9E86/5F6DDF02/5F6A66A6" Ref="#PWR056"  Part="1"
 AR Path="/5F4A9E86/5F60074F/5F6A66A6" Ref="#PWR?"  Part="1"
-F 0 "#PWR035" H 6750 4150 50  0001 C CNN
+F 0 "#PWR056" H 6750 4150 50  0001 C CNN
 F 1 "GND" H 6755 4227 50  0000 C CNN
 F 2 "" H 6750 4400 50  0001 C CNN
@@
 AR Path="/5F4A9E86/5F6DDF02/5F6A7DE8" Ref="#PWR054"  Part="1"
 AR Path="/5F4A9E86/5F60074F/5F6A7DE8" Ref="#PWR?"  Part="1"
-F 0 "#PWR033" H 6300 4150 50  0001 C CNN
+F 0 "#PWR054" H 6300 4150 50  0001 C CNN
 F 1 "GND" H 6305 4227 50  0000 C CNN
 F 2 "" H 6300 4400 50  0001 C CNN
@@
 AR Path="/5F4A9E86/5F6DDF02/5F6B5A68" Ref="#PWR051"  Part="1"
 AR Path="/5F4A9E86/5F60074F/5F6B5A68" Ref="#PWR?"  Part="1"
-F 0 "#PWR030" H 4450 4150 50  0001 C CNN
+F 0 "#PWR051" H 4450 4150 50  0001 C CNN
 F 1 "GND" H 4455 4227 50  0000 C CNN
 F 2 "" H 4450 4400 50  0001 C CNN
@@
 AR Path="/5F4A9E86/5F6DDF02/5F6B8BDC" Ref="C15"  Part="1"
 AR Path="/5F4A9E86/5F60074F/5F6B8BDC" Ref="C?"  Part="1"
-F 0 "C6" H 4215 4146 50  0000 L CNN
+F 0 "C15" H 4215 4146 50  0000 L CNN
 F 1 "10n" H 4215 4055 50  0000 L CNN
 F 2 "Capacitor_SMD:C_0402_1005Metric" H 4138 3950 50  0001 C CNN
@@
 AR Path="/5F4A9E86/5F6DDF02/5F6B95E0" Ref="C16"  Part="1"
 AR Path="/5F4A9E86/5F60074F/5F6B95E0" Ref="C?"  Part="1"
-F 0 "C7" H 4565 4146 50  0000 L CNN
+F 0 "C16" H 4565 4146 50  0000 L CNN
 F 1 "10n" H 4565 4055 50  0000 L CNN
 F 2 "Capacitor_SMD:C_0402_1005Metric" H 4488 3950 50  0001 C CNN
@@
 AR Path="/5F4A9E86/5F6DDF02/5F6B50D9" Ref="#PWR050"  Part="1"
 AR Path="/5F4A9E86/5F60074F/5F6B50D9" Ref="#PWR?"  Part="1"
-F 0 "#PWR029" H 4100 4150 50  0001 C CNN
+F 0 "#PWR050" H 4100 4150 50  0001 C CNN
 F 1 "GND" H 4105 4227 50  0000 C CNN
 F 2 "" H 4100 4400 50  0001 C CNN
@@
 AR Path="/5F4A9E86/5F64E559/5FA5F61A" Ref="#PWR038"  Part="1"
 AR Path="/5F4A9E86/5F64E7E9/5FA5F61A" Ref="#PWR045"  Part="1"
-F 0 "#PWR031" H 5100 3100 50  0001 C CNN
+F 0 "#PWR052" H 5100 3100 50  0001 C CNN
 F 1 "+3V3" H 5115 3423 50  0000 C CNN
 F 2 "" H 5100 3250 50  0001 C CNN
@@
 AR Path="/5F4A9E86/5F64E559/5FA5FB6F" Ref="#PWR039"  Part="1"
 AR Path="/5F4A9E86/5F64E7E9/5FA5FB6F" Ref="#PWR046"  Part="1"
-F 0 "#PWR032" H 5450 3100 50  0001 C CNN
+F 0 "#PWR053" H 5450 3100 50  0001 C CNN
 F 1 "+3V3" H 5465 3423 50  0000 C CNN
 F 2 "" H 5450 3250 50  0001 C CNN
@@
 AR Path="/5F4A9E86/5F64E559/5FA5FD7B" Ref="#PWR041"  Part="1"
 AR Path="/5F4A9E86/5F64E7E9/5FA5FD7B" Ref="#PWR048"  Part="1"
-F 0 "#PWR034" H 6750 3150 50  0001 C CNN
+F 0 "#PWR055" H 6750 3150 50  0001 C CNN
 F 1 "+3V3" H 6765 3473 50  0000 C CNN
 F 2 "" H 6750 3300 50  0001 C CNN
@@
 AR Path="/5F4A9E86/5F64E7E9/5FF1EA9B" Ref="R52"  Part="1"
 AR Path="/5F4A9E86/5F6DDF02/5FF1EA9B" Ref="R58"  Part="1"
-F 0 "R40" V 4593 3700 50  0000 C CNN
-F 1 "10K" V 4684 3700 50  0000 C CNN
+F 0 "R58" V 4593 3700 50  0000 C CNN
+F 1 "10k" V 4684 3700 50  0000 C CNN
 F 2 "Resistor_SMD:R_0402_1005Metric" V 4730 3700 50  0001 C CNN
 F 3 "~" H 4800 3700 50  0001 C CNN
+F 4 "RMCF0402FT10K0CT-ND" H 4800 3700 50  0001 C CNN "Digikey"
+F 5 "RMCF0402FT10K0" H 4800 3700 50  0001 C CNN "MPN"
+F 6 "Stackpole" H 4800 3700 50  0001 C CNN "Manufacturer"
 	1    4800 3700
 	0    1    1    0
@@
 AR Path="/5F4A9E86/5F64E7E9/5FF1F393" Ref="R53"  Part="1"
 AR Path="/5F4A9E86/5F6DDF02/5FF1F393" Ref="R59"  Part="1"
-F 0 "R41" V 4593 3900 50  0000 C CNN
-F 1 "10K" V 4684 3900 50  0000 C CNN
+F 0 "R59" V 4593 3900 50  0000 C CNN
+F 1 "10k" V 4684 3900 50  0000 C CNN
 F 2 "Resistor_SMD:R_0402_1005Metric" V 4730 3900 50  0001 C CNN
 F 3 "~" H 4800 3900 50  0001 C CNN
+F 4 "RMCF0402FT10K0CT-ND" H 4800 3900 50  0001 C CNN "Digikey"
+F 5 "RMCF0402FT10K0" H 4800 3900 50  0001 C CNN "MPN"
+F 6 "Stackpole" H 4800 3900 50  0001 C CNN "Manufacturer"
 	1    4800 3900
 	0    1    1    0
@@
 AR Path="/5F4A9E86/5F64E7E9/5FF1F59B" Ref="R54"  Part="1"
 AR Path="/5F4A9E86/5F6DDF02/5FF1F59B" Ref="R60"  Part="1"
-F 0 "R42" H 5030 3354 50  0000 R CNN
-F 1 "10K" H 5030 3445 50  0000 R CNN
+F 0 "R60" H 5030 3354 50  0000 R CNN
+F 1 "10k" H 5030 3445 50  0000 R CNN
 F 2 "Resistor_SMD:R_0402_1005Metric" V 5030 3400 50  0001 C CNN
 F 3 "~" H 5100 3400 50  0001 C CNN
+F 4 "RMCF0402FT10K0CT-ND" H 5100 3400 50  0001 C CNN "Digikey"
+F 5 "RMCF0402FT10K0" H 5100 3400 50  0001 C CNN "MPN"
+F 6 "Stackpole" H 5100 3400 50  0001 C CNN "Manufacturer"
 	1    5100 3400
 	-1   0    0    1
@@
 AR Path="/5F4A9E86/5F64E7E9/5FF1F8A9" Ref="R55"  Part="1"
 AR Path="/5F4A9E86/5F6DDF02/5FF1F8A9" Ref="R61"  Part="1"
-F 0 "R43" H 5380 3354 50  0000 R CNN
-F 1 "10K" H 5380 3445 50  0000 R CNN
+F 0 "R61" H 5380 3354 50  0000 R CNN
+F 1 "10k" H 5380 3445 50  0000 R CNN
 F 2 "Resistor_SMD:R_0402_1005Metric" V 5380 3400 50  0001 C CNN
 F 3 "~" H 5450 3400 50  0001 C CNN
+F 4 "RMCF0402FT10K0CT-ND" H 5450 3400 50  0001 C CNN "Digikey"
+F 5 "RMCF0402FT10K0" H 5450 3400 50  0001 C CNN "MPN"
+F 6 "Stackpole" H 5450 3400 50  0001 C CNN "Manufacturer"
 	1    5450 3400
 	-1   0    0    1
@@
 AR Path="/5F4A9E86/5F64E7E9/5FF1FAB4" Ref="R56"  Part="1"
 AR Path="/5F4A9E86/5F6DDF02/5FF1FAB4" Ref="R62"  Part="1"
-F 0 "R44" V 6707 3700 50  0000 C CNN
-F 1 "10K" V 6616 3700 50  0000 C CNN
+F 0 "R62" V 6707 3700 50  0000 C CNN
+F 1 "10k" V 6616 3700 50  0000 C CNN
 F 2 "Resistor_SMD:R_0402_1005Metric" V 6430 3700 50  0001 C CNN
 F 3 "~" H 6500 3700 50  0001 C CNN
+F 4 "RMCF0402FT10K0CT-ND" H 6500 3700 50  0001 C CNN "Digikey"
+F 5 "RMCF0402FT10K0" H 6500 3700 50  0001 C CNN "MPN"
+F 6 "Stackpole" H 6500 3700 50  0001 C CNN "Manufacturer"
 	1    6500 3700
 	0    -1   -1   0
@@
 AR Path="/5F4A9E86/5F64E7E9/5FF1FD2A" Ref="R57"  Part="1"
 AR Path="/5F4A9E86/5F6DDF02/5FF1FD2A" Ref="R63"  Part="1"
-F 0 "R45" H 6820 3496 50  0000 L CNN
-F 1 "10K" H 6820 3405 50  0000 L CNN
+F 0 "R63" H 6820 3496 50  0000 L CNN
+F 1 "10k" H 6820 3405 50  0000 L CNN
 F 2 "Resistor_SMD:R_0402_1005Metric" V 6680 3450 50  0001 C CNN
 F 3 "~" H 6750 3450 50  0001 C CNN
+F 4 "RMCF0402FT10K0CT-ND" H 6750 3450 50  0001 C CNN "Digikey"
+F 5 "RMCF0402FT10K0" H 6750 3450 50  0001 C CNN "MPN"
+F 6 "Stackpole" H 6750 3450 50  0001 C CNN "Manufacturer"
 	1    6750 3450
 	1    0    0    -1
@@
 AR Path="/5F4A9E86/5F6DDF02/5FC19961" Ref="#PWR0148"  Part="1"
 AR Path="/5F4A9E86/5F60074F/5FC19961" Ref="#PWR?"  Part="1"
-F 0 "#PWR0145" H 5550 3550 50  0001 C CNN
+F 0 "#PWR0148" H 5550 3550 50  0001 C CNN
 F 1 "GND" H 5555 3627 50  0000 C CNN
 F 2 "" H 5550 3800 50  0001 C CNN
