File: PCB/Power.sch (KiCad schematic (older format))
At the start: 26 parts, among them J8 Barrel_Jack_Switch, Q1 FDN338P, Q2 MMBT3904, Q3 FDN338P, U7 DMP1005UFDF, U8 AP2114HA-3.3TRG1

Commit message: PCB Version 1: As Sent to Fab
Parts:
- C34: Digikey 311-4046-1-ND -> 587-1243-1-ND; MPN CC0603KRX5R9BB104 -> UMK107B7104KA-T; Manufacturer Yageo -> Taiyo Yuden
- C37: value 4.7uF -> 10uF; Digikey 1276-1055-1-ND -> 732-865081745005CT-ND; MPN CL31B475KAHNNNE -> 865081745005; Manufacturer Samsung -> Würth Elektronik
- D13: value LED -> LED_Red; Digikey (none) -> 160-1447-1-ND; MPN (none) -> LTST-C191KRKT; Manufacturer (none) -> Lite-On Inc.
- D14: Digikey (none) -> S4SCT-ND
- D15: value LED -> LED_Green; Digikey (none) -> 160-1446-1-ND; MPN (none) -> LTST-C191KGKT; Manufacturer (none) -> Lite-On Inc.
- D16: value LED -> LED_Blue; Digikey (none) -> 160-1647-1-ND; MPN (none) -> LTST-C191TBKT; Manufacturer (none) -> Lite-On Inc.
- R21: Digikey (none) -> RMCF0402FT510KCT-ND; MPN (none) -> RMCF0402FT510K; Manufacturer (none) -> Stackpole
- R22, R29, R30: Digikey (none) -> RMCF0402FT1K00CT-ND; MPN (none) -> RMCF0402FT1K00; Manufacturer (none) -> Stackpole
- R23: Digikey (none) -> RMCF0402FT4K70CT-ND; MPN (none) -> RMCF0402FT4K70; Manufacturer (none) -> Stackpole
- R24, R25, R26: Digikey (none) -> 311-270JRCT-ND; MPN (none) -> RC0402JR-07270RL; Manufacturer (none) -> Yageo
- R27: Digikey (none) -> RMCF0402ZT0R00CT-ND; MPN (none) -> RMCF0402ZT0R00; Manufacturer (none) -> Stackpole
- U7: Digikey (none) -> DMP1005UFDF-7DICT-ND
Changed lines of the file:
@@
 F 2 "Capacitor_SMD:C_0603_1608Metric" H 3188 3250 50  0001 C CNN
 F 3 "~" H 3150 3400 50  0001 C CNN
-F 4 "311-4046-1-ND" H 3150 3400 50  0001 C CNN "Digikey"
-F 5 "CC0603KRX5R9BB104" H 3150 3400 50  0001 C CNN "MPN"
-F 6 "Yageo" H 3150 3400 50  0001 C CNN "Manufacturer"
+F 4 "587-1243-1-ND" H 3150 3400 50  0001 C CNN "Digikey"
+F 5 "UMK107B7104KA-T" H 3150 3400 50  0001 C CNN "MPN"
+F 6 "Taiyo Yuden" H 3150 3400 50  0001 C CNN "Manufacturer"
 	1    3150 3400
 	1    0    0    -1
@@
 F 2 "Resistor_SMD:R_0402_1005Metric" V 3480 3600 50  0001 C CNN
 F 3 "~" H 3550 3600 50  0001 C CNN
+F 4 "RMCF0402FT1K00CT-ND" H 3550 3600 50  0001 C CNN "Digikey"
+F 5 "RMCF0402FT1K00" H 3550 3600 50  0001 C CNN "MPN"
+F 6 "Stackpole" H 3550 3600 50  0001 C CNN "Manufacturer"
 	1    3550 3600
 	1    0    0    -1
@@
 F 2 "Diode_SMD:D_SMB_Modified" V 4050 3300 50  0001 C CNN
 F 3 "~" V 4050 3300 50  0001 C CNN
+F 4 "S4SCT-ND" H 4050 3300 50  0001 C CNN "Digikey"
 	1    4050 3300
 	1    0    0    -1
@@
 F 2 "Resistor_SMD:R_0402_1005Metric" V 3480 5300 50  0001 C CNN
 F 3 "~" H 3550 5300 50  0001 C CNN
+F 4 "RMCF0402FT4K70CT-ND" H 3550 5300 50  0001 C CNN "Digikey"
+F 5 "RMCF0402FT4K70" H 3550 5300 50  0001 C CNN "MPN"
+F 6 "Stackpole" H 3550 5300 50  0001 C CNN "Manufacturer"
 	1    3550 5300
 	0    -1   -1   0
@@
 F 2 "Resistor_SMD:R_0402_1005Metric" V 3080 5300 50  0001 C CNN
 F 3 "~" H 3150 5300 50  0001 C CNN
+F 4 "RMCF0402FT510KCT-ND" H 3150 5300 50  0001 C CNN "Digikey"
+F 5 "RMCF0402FT510K" H 3150 5300 50  0001 C CNN "MPN"
+F 6 "Stackpole" H 3150 5300 50  0001 C CNN "Manufacturer"
 	1    3150 5300
 	0    -1   -1   0
@@
 AR Path="/5F8D38D7" Ref="U?"  Part="1"
 AR Path="/5F8CC9DA/5F8D38D7" Ref="U7"  Part="1"
+AR Path="/5F4A9E86/5F8D38D7" Ref="U7"  Part="1"
 F 0 "U7" V 4742 2950 50  0000 C CNN
 F 1 "DMP1005UFDF" V 4651 2950 50  0000 C CNN
 F 2 "Package_DFN_QFN:Diodes_UDFN2020-6_Type-F" H 4500 2950 50  0001 C CNN
 F 3 "" H 4500 2950 50  0001 C CNN
+F 4 "DMP1005UFDF-7DICT-ND" H 4500 2950 50  0001 C CNN "Digikey"
 	1    4500 2950
 	0    1    -1   0
@@
 F 2 "Resistor_SMD:R_0402_1005Metric" V 7230 3950 50  0001 C CNN
 F 3 "~" H 7300 3950 50  0001 C CNN
+F 4 "RMCF0402ZT0R00CT-ND" H 7300 3950 50  0001 C CNN "Digikey"
+F 5 "RMCF0402ZT0R00" H 7300 3950 50  0001 C CNN "MPN"
+F 6 "Stackpole" H 7300 3950 50  0001 C CNN "Manufacturer"
 	1    7300 3950
 	0    1    1    0
@@
 F 2 "Resistor_SMD:R_0402_1005Metric" V 7230 4650 50  0001 C CNN
 F 3 "~" H 7300 4650 50  0001 C CNN
+F 4 "RMCF0402FT1K00CT-ND" H 7300 4650 50  0001 C CNN "Digikey"
+F 5 "RMCF0402FT1K00" H 7300 4650 50  0001 C CNN "MPN"
+F 6 "Stackpole" H 7300 4650 50  0001 C CNN "Manufacturer"
 	1    7300 4650
 	0    1    1    0
@@
 F 2 "Resistor_SMD:R_0402_1005Metric" V 7780 4150 50  0001 C CNN
 F 3 "~" H 7850 4150 50  0001 C CNN
+F 4 "RMCF0402FT1K00CT-ND" H 7850 4150 50  0001 C CNN "Digikey"
+F 5 "RMCF0402FT1K00" H 7850 4150 50  0001 C CNN "MPN"
+F 6 "Stackpole" H 7850 4150 50  0001 C CNN "Manufacturer"
 	1    7850 4150
 	-1   0    0    1
@@
 F 2 "Resistor_SMD:R_0402_1005Metric" V 3730 1550 50  0001 C CNN
 F 3 "~" H 3800 1550 50  0001 C CNN
+F 4 "311-270JRCT-ND" H 3800 1550 50  0001 C CNN "Digikey"
+F 5 "RC0402JR-07270RL" H 3800 1550 50  0001 C CNN "MPN"
+F 6 "Yageo" H 3800 1550 50  0001 C CNN "Manufacturer"
 	1    3800 1550
 	-1   0    0    1
@@
 P 3800 1850
 F 0 "D13" V 3839 1732 50  0000 R CNN
-F 1 "LED" V 3748 1732 50  0000 R CNN
+F 1 "LED_Red" V 3748 1732 50  0000 R CNN
 F 2 "LED_SMD:LED_0603_1608Metric" H 3800 1850 50  0001 C CNN
 F 3 "~" H 3800 1850 50  0001 C CNN
+F 4 "160-1447-1-ND" H 3800 1850 50  0001 C CNN "Digikey"
+F 5 "LTST-C191KRKT" H 3800 1850 50  0001 C CNN "MPN"
+F 6 "Lite-On Inc." H 3800 1850 50  0001 C CNN "Manufacturer"
 	1    3800 1850
 	0    -1   -1   0
@@
 F 2 "Resistor_SMD:R_0402_1005Metric" V 4080 1550 50  0001 C CNN
 F 3 "~" H 4150 1550 50  0001 C CNN
+F 4 "311-270JRCT-ND" H 4150 1550 50  0001 C CNN "Digikey"
+F 5 "RC0402JR-07270RL" H 4150 1550 50  0001 C CNN "MPN"
+F 6 "Yageo" H 4150 1550 50  0001 C CNN "Manufacturer"
 	1    4150 1550
 	-1   0    0    1
@@
 P 4150 1850
 F 0 "D15" V 4189 1732 50  0000 R CNN
-F 1 "LED" V 4098 1732 50  0000 R CNN
+F 1 "LED_Green" V 4098 1732 50  0000 R CNN
 F 2 "LED_SMD:LED_0603_1608Metric" H 4150 1850 50  0001 C CNN
 F 3 "~" H 4150 1850 50  0001 C CNN
+F 4 "160-1446-1-ND" H 4150 1850 50  0001 C CNN "Digikey"
+F 5 "LTST-C191KGKT" H 4150 1850 50  0001 C CNN "MPN"
+F 6 "Lite-On Inc." H 4150 1850 50  0001 C CNN "Manufacturer"
 	1    4150 1850
 	0    -1   -1   0
@@
 F 2 "Resistor_SMD:R_0402_1005Metric" V 4430 1550 50  0001 C CNN
 F 3 "~" H 4500 1550 50  0001 C CNN
+F 4 "311-270JRCT-ND" H 4500 1550 50  0001 C CNN "Digikey"
+F 5 "RC0402JR-07270RL" H 4500 1550 50  0001 C CNN "MPN"
+F 6 "Yageo" H 4500 1550 50  0001 C CNN "Manufacturer"
 	1    4500 1550
 	-1   0    0    1
@@
 P 4500 1850
 F 0 "D16" V 4539 1732 50  0000 R CNN
-F 1 "LED" V 4448 1732 50  0000 R CNN
+F 1 "LED_Blue" V 4448 1732 50  0000 R CNN
 F 2 "LED_SMD:LED_0603_1608Metric" H 4500 1850 50  0001 C CNN
 F 3 "~" H 4500 1850 50  0001 C CNN
+F 4 "160-1647-1-ND" H 4500 1850 50  0001 C CNN "Digikey"
+F 5 "LTST-C191TBKT" H 4500 1850 50  0001 C CNN "MPN"
+F 6 "Lite-On Inc." H 4500 1850 50  0001 C CNN "Manufacturer"
 	1    4500 1850
 	0    -1   -1   0
@@
 AR Path="/5F8CC9DA/5FBAEF90" Ref="C37"  Part="1"
 F 0 "C37" H 7365 1946 50  0000 L CNN
-F 1 "4.7uF" H 7365 1855 50  0000 L CNN
+F 1 "10uF" H 7365 1855 50  0000 L CNN
 F 2 "Capacitor_THT:CP_Radial_D6.3mm_P2.50mm" H 7288 1750 50  0001 C CNN
 F 3 "~" H 7250 1900 50  0001 C CNN
-F 4 "1276-1055-1-ND" H 7250 1900 50  0001 C CNN "Digikey"
-F 5 "Samsung" H 7250 1900 50  0001 C CNN "Manufacturer"
-F 6 "CL31B475KAHNNNE" H 7250 1900 50  0001 C CNN "MPN"
+F 4 "732-865081745005CT-ND" H 7250 1900 50  0001 C CNN "Digikey"
+F 5 "Würth Elektronik" H 7250 1900 50  0001 C CNN "Manufacturer"
+F 6 "865081745005" H 7250 1900 50  0001 C CNN "MPN"
 	1    7250 1900
 	1    0    0    -1
