File: PCB/QuadEncoder.sch (KiCad schematic (older format))
At the start: 8 parts

Commit message: Schematic, Code Refactor, 328P workspace
Parts:
- removed C? (x2): 10n, symbol Device:C
- removed R? (x2): 10k, symbol Device:R
- removed R? (x2): 10K, symbol Device:R
- removed SW?: Rotary_Encoder_Switch, symbol Device:Rotary_Encoder_Switch
- added C10, C9: 12pF, symbol Device:C_Small
- added C11, C8: 1uF, symbol Device:C_Small
- added C7: 0.1uF, symbol Device:C_Small
- added D1: LED, symbol Device:LED
- added J3: Programming Header, symbol Connector_Generic:Conn_02x03_Odd_Even
- added J4: UART, symbol Connector_Generic:Conn_01x02
- added JP3: SolderJumper_2_Open, symbol Jumper:SolderJumper_2_Open
- added R10, R11, R14, R15, R4, R5, R6, R7: 10k, symbol Device:R
- added R12, R13, R16, R17, R8, R9: 270R, symbol Device:R
- added RV1, RV2, RV3: R_POT, symbol Device:R_POT
- added SW2, SW3, SW4, SW5, SW6, SW7: SW_Push_LED, symbol Switch:SW_Push_LED
- added TP1: TestPoint, symbol Connector:TestPoint
- added U5: MCP23017_SO, Package_SO:SOIC-28W_7.5x17.9mm_P1.27mm, symbol Interface_Expansion:MCP23017_SO
- added Y1: 16MHz, symbol Device:Crystal_Small
- gave numbers to parts that had none: 1
Connections:
- net labels added: BTN_PRESSED, CIDO, CODI, ENC1_A, ENC1_B, ENC1_SW, ENC2_A, ENC2_B, ENC2_SW, ENC3_A, ENC3_B, ENC3_SW, ENC4_A, ENC4_B, ENC4_SW, INTA, LED, LED_Power, RXD, SCL, SCLK, SDA, SLD1, SLD2, SLD3, SPARE, SW_1, SW_2, SW_3, SW_4, SW_5, SW_6, TXD, XTAL1, XTAL2, ~RESET
- wire segments 16 -> 169
- no-connect marks 0 -> 7
Other:
- note added: "ATMega Aux Processor"
- note added: "Encoders x4"
- note added: "Faders x3"
- note added: "INT Pins Mirrored\nIOCON:MIRROR = 1"
- note added: "IO Expander\nfor Encoder and Keypad Switches"
- note added: "Keypad Switches x6"
- moved on the sheet: U4

Commit message: WIP PCB changes
Parts:
- removed C10, C9: 12pF, symbol Device:C_Small
- removed R10, R11, R14, R15, R6, R7: 10k, symbol Device:R
- removed Y1: 16MHz, symbol Device:Crystal_Small
- added C3, C4: 20p, Capacitor_SMD:C_0402_1005Metric, symbol Device:C_Small
- added D2, D3, D4, D5, D6, D7: LED_CoolWhite, symbol Device:LED
- added R34, R35, R36, R37, R38, R39: 10K, Resistor_SMD:R_0402_1005Metric, symbol Device:R
- added Y1: 16MHz, MK_Library:ECS-120-12-36-AGN, symbol Device:Crystal_GND2_Small
- C1: renamed from C7; footprint (none) -> Capacitor_SMD:C_0603_1608Metric; Digikey (none) -> 311-4046-1-ND; MPN (none) -> CC0603KRX5R9BB104; Manufacturer (none) -> Yageo
- C2: renamed from C8; footprint (none) -> Capacitor_SMD:C_0603_1608Metric; Digikey (none) -> 1276-1102-1-ND; MPN (none) -> CL10A105KA8NNNC; Manufacturer (none) -> Samsung
- C5: renamed from C11; footprint (none) -> Capacitor_SMD:C_0603_1608Metric; Digikey (none) -> 1276-1102-1-ND; MPN (none) -> CL10A105KA8NNNC; Manufacturer (none) -> Samsung
- D1: footprint (none) -> LED_SMD:LED_0603_1608Metric; Digikey (none) -> 160-1446-1-ND; MPN (none) -> LTST-C191KGKT; Manufacturer (none) -> Lite-On Inc.
- J1: renamed from J3; footprint (none) -> Connector_PinHeader_2.54mm:PinHeader_2x03_P2.54mm_Vertical; Digikey (none) -> 2057-PH2-06-UA-ND; MPN (none) -> PH2-06-UA; Manufacturer (none) -> Adam Tech
- J2: renamed from J4; footprint (none) -> Connector_PinHeader_2.54mm:PinHeader_1x02_P2.54mm_Vertical
- JP1: renamed from JP3; footprint (none) -> Jumper:SolderJumper-2_P1.3mm_Open_Pad1.0x1.5mm
- R1: renamed from R4; value 10k -> 270R; footprint (none) -> Resistor_SMD:R_0402_1005Metric; Digikey (none) -> 311-270JRCT-ND; MPN (none) -> RC0402JR-07270RL; Manufacturer (none) -> Yageo
- R2: renamed from R5; footprint (none) -> Resistor_SMD:R_0402_1005Metric; Digikey (none) -> RMCF0402FT10K0CT-ND; MPN (none) -> RMCF0402FT10K0; Manufacturer (none) -> Stackpole
- R3: renamed from R8; footprint (none) -> Resistor_SMD:R_0402_1005Metric; Digikey (none) -> 311-270JRCT-ND; MPN (none) -> RC0402JR-07270RL; Manufacturer (none) -> Yageo
- R4: renamed from R9; footprint (none) -> Resistor_SMD:R_0402_1005Metric; Digikey (none) -> 311-270JRCT-ND; MPN (none) -> RC0402JR-07270RL; Manufacturer (none) -> Yageo
- R5: renamed from R12; footprint (none) -> Resistor_SMD:R_0402_1005Metric; Digikey (none) -> 311-270JRCT-ND; MPN (none) -> RC0402JR-07270RL; Manufacturer (none) -> Yageo
- R6: renamed from R13; footprint (none) -> Resistor_SMD:R_0402_1005Metric; Digikey (none) -> 311-270JRCT-ND; MPN (none) -> RC0402JR-07270RL; Manufacturer (none) -> Yageo
- R7: renamed from R16; footprint (none) -> Resistor_SMD:R_0402_1005Metric; Digikey (none) -> 311-270JRCT-ND; MPN (none) -> RC0402JR-07270RL; Manufacturer (none) -> Yageo
- R8: renamed from R17; footprint (none) -> Resistor_SMD:R_0402_1005Metric; Digikey (none) -> 311-270JRCT-ND; MPN (none) -> RC0402JR-07270RL; Manufacturer (none) -> Yageo
- RV1, RV2, RV3: footprint (none) -> EMRSNxEOS:SliderHeader; Digikey (none) -> PTA4553-2210CIB103-ND; MPN (none) -> PTA4553-2210CIB103; Manufacturer (none) -> Bourns Inc.
- SW1: renamed from SW2; footprint (none) -> MK_Library:SW_Cherry_MX_Single_LED; Digikey (none) -> CH160-ND; MPN (none) -> MX1A-11NW; Manufacturer (none) -> Cherry Americas LLC
- SW2: renamed from SW3; footprint (none) -> MK_Library:SW_Cherry_MX_Single_LED; Digikey (none) -> CH160-ND; MPN (none) -> MX1A-11NW; Manufacturer (none) -> Cherry Americas LLC
- SW3: renamed from SW4; footprint (none) -> MK_Library:SW_Cherry_MX_Single_LED; Digikey (none) -> CH160-ND; MPN (none) -> MX1A-11NW; Manufacturer (none) -> Cherry Americas LLC
- SW4: renamed from SW5; footprint (none) -> MK_Library:SW_Cherry_MX_Single_LED; Digikey (none) -> CH160-ND; MPN (none) -> MX1A-11NW; Manufacturer (none) -> Cherry Americas LLC
- SW5: renamed from SW6; footprint (none) -> MK_Library:SW_Cherry_MX_Single_LED; Digikey (none) -> CH160-ND; MPN (none) -> MX1A-11NW; Manufacturer (none) -> Cherry Americas LLC
- SW6: renamed from SW7; footprint (none) -> MK_Library:SW_Cherry_MX_Single_LED; Digikey (none) -> CH160-ND; MPN (none) -> MX1A-11NW; Manufacturer (none) -> Cherry Americas LLC
- TP1: footprint (none) -> TestPoint:TestPoint_Pad_1.5x1.5mm
- U1: renamed from U4; footprint Package_DIP:DIP-28_W7.62mm -> Package_QFP:TQFP-32_7x7mm_P0.8mm; Digikey (none) -> ATMEGA328PB-AU-ND; MPN (none) -> ATMEGA328PB-AU; Manufacturer (none) -> Atmel
- U2: renamed from U5; Digikey (none) -> MCP23017T-E/SOCT-ND; MPN (none) -> MCP23017T-E/SO; Manufacturer (none) -> Microchip Technology
Connections:
- net +3V3: now also R34.1, R35.1, R36.1, R37.1, R38.1, R39.1
- net ENC1_A: now also U1.13 (PD7); no longer U1.2 (PD0)
- net ENC1_B: now also U1.12 (PD6); no longer U1.3 (PD1)
- net ENC1_SW: now also U2.4 (GPB3); no longer U2.21 (GPA0)
- net ENC2_A: now also U1.11 (PD5); no longer U1.4 (PD2)
- net ENC2_B: now also U1.6 (PD4); no longer U1.5 (PD3)
- net ENC2_SW: now also U2.3 (GPB2); no longer U2.22 (GPA1)
- net ENC3_A: now also U1.5 (PD3); no longer U1.6 (PD4)
- net ENC3_B: now also U1.4 (PD2); no longer U1.11 (PD5)
- net ENC3_SW: now also U2.2 (GPB1); no longer U2.23 (GPA2)
- net ENC4_A: now also U1.3 (PD1); no longer U1.12 (PD6)
- net ENC4_B: now also U1.2 (PD0); no longer U1.13 (PD7)
- net ENC4_SW: now also U2.1 (GPB0); no longer U2.24 (GPA3)
- net GND: now also C3.1, C4.1, Y1.2
- net SLD1: now also U1.25 (PC2); no longer U1.23 (PC0)
- net SLD3: now also U1.23 (PC0); no longer U1.25 (PC2)
- net SW_1: now also U2.26 (GPA5), R34.2; no longer U2.1 (GPB0)
- net SW_2: now also SW2.2, U2.25 (GPA4), R35.2; no longer SW3.2, U2.2 (GPB1)
- net SW_3: now also SW3.2, U2.24 (GPA3), R36.2; no longer SW5.2, U2.3 (GPB2)
- net SW_4: now also SW4.2, U2.21 (GPA0), R37.2; no longer SW2.2, U2.4 (GPB3)
- net SW_5: now also SW5.2, U2.22 (GPA1), R38.2; no longer SW4.2, U2.5 (GPB4)
- net SW_6: now also U2.23 (GPA2), R39.2; no longer U2.6 (GPB5)
- net XTAL1: now also C3.2, Y1.1
- net XTAL2: now also C4.2, Y1.3
- no-connect marks 7 -> 19
Other:
- note added: "All encoders on the same port to\nfacilitate fast channel reading upon\nPin Change Interrupt (PCINT)"
- note added: "Switch LEDs for BOM"
- note added: "Talks directly to Core Processor, not Aux Processor"

Commit message: PCB Version 1: As Sent to Fab
Parts:
- C1: Digikey 311-4046-1-ND -> 587-1243-1-ND; MPN CC0603KRX5R9BB104 -> UMK107B7104KA-T; Manufacturer Yageo -> Taiyo Yuden
- D1: value LED -> LED_Green
- R34, R35, R36, R37, R38, R39: value 10K -> 10k; Digikey (none) -> RMCF0402FT10K0CT-ND; MPN (none) -> RMCF0402FT10K0; Manufacturer (none) -> Stackpole
Changed lines of the file:
@@
 F 2 "Capacitor_SMD:C_0603_1608Metric" H 2750 2850 50  0001 C CNN
 F 3 "~" H 2750 2850 50  0001 C CNN
-F 4 "311-4046-1-ND" H 2750 2850 50  0001 C CNN "Digikey"
-F 5 "CC0603KRX5R9BB104" H 2750 2850 50  0001 C CNN "MPN"
-F 6 "Yageo" H 2750 2850 50  0001 C CNN "Manufacturer"
+F 4 "587-1243-1-ND" H 2750 2850 50  0001 C CNN "Digikey"
+F 5 "UMK107B7104KA-T" H 2750 2850 50  0001 C CNN "MPN"
+F 6 "Taiyo Yuden" H 2750 2850 50  0001 C CNN "Manufacturer"
 	1    2750 2850
 	1    0    0    -1
@@
 P 4300 8200
 F 0 "D1" V 4339 8083 50  0000 R CNN
-F 1 "LED" V 4248 8083 50  0000 R CNN
+F 1 "LED_Green" V 4248 8083 50  0000 R CNN
 F 2 "LED_SMD:LED_0603_1608Metric" H 4300 8200 50  0001 C CNN
 F 3 "~" H 4300 8200 50  0001 C CNN
@@
 P 8450 4750
 F 0 "R34" H 8520 4796 50  0000 L CNN
-F 1 "10K" H 8520 4705 50  0000 L CNN
+F 1 "10k" H 8520 4705 50  0000 L CNN
 F 2 "Resistor_SMD:R_0402_1005Metric" V 8380 4750 50  0001 C CNN
 F 3 "~" H 8450 4750 50  0001 C CNN
+F 4 "RMCF0402FT10K0CT-ND" H 8450 4750 50  0001 C CNN "Digikey"
+F 5 "RMCF0402FT10K0" H 8450 4750 50  0001 C CNN "MPN"
+F 6 "Stackpole" H 8450 4750 50  0001 C CNN "Manufacturer"
 	1    8450 4750
 	1    0    0    -1
@@
 P 10900 4750
 F 0 "R36" H 10970 4796 50  0000 L CNN
-F 1 "10K" H 10970 4705 50  0000 L CNN
+F 1 "10k" H 10970 4705 50  0000 L CNN
 F 2 "Resistor_SMD:R_0402_1005Metric" V 10830 4750 50  0001 C CNN
 F 3 "~" H 10900 4750 50  0001 C CNN
+F 4 "RMCF0402FT10K0CT-ND" H 10900 4750 50  0001 C CNN "Digikey"
+F 5 "RMCF0402FT10K0" H 10900 4750 50  0001 C CNN "MPN"
+F 6 "Stackpole" H 10900 4750 50  0001 C CNN "Manufacturer"
 	1    10900 4750
 	1    0    0    -1
@@
 P 13200 4750
 F 0 "R38" H 13270 4796 50  0000 L CNN
-F 1 "10K" H 13270 4705 50  0000 L CNN
+F 1 "10k" H 13270 4705 50  0000 L CNN
 F 2 "Resistor_SMD:R_0402_1005Metric" V 13130 4750 50  0001 C CNN
 F 3 "~" H 13200 4750 50  0001 C CNN
+F 4 "RMCF0402FT10K0CT-ND" H 13200 4750 50  0001 C CNN "Digikey"
+F 5 "RMCF0402FT10K0" H 13200 4750 50  0001 C CNN "MPN"
+F 6 "Stackpole" H 13200 4750 50  0001 C CNN "Manufacturer"
 	1    13200 4750
 	1    0    0    -1
@@
 P 13200 5950
 F 0 "R39" H 13270 5996 50  0000 L CNN
-F 1 "10K" H 13270 5905 50  0000 L CNN
+F 1 "10k" H 13270 5905 50  0000 L CNN
 F 2 "Resistor_SMD:R_0402_1005Metric" V 13130 5950 50  0001 C CNN
 F 3 "~" H 13200 5950 50  0001 C CNN
+F 4 "RMCF0402FT10K0CT-ND" H 13200 5950 50  0001 C CNN "Digikey"
+F 5 "RMCF0402FT10K0" H 13200 5950 50  0001 C CNN "MPN"
+F 6 "Stackpole" H 13200 5950 50  0001 C CNN "Manufacturer"
 	1    13200 5950
 	1    0    0    -1
@@
 P 10900 5950
 F 0 "R37" H 10970 5996 50  0000 L CNN
-F 1 "10K" H 10970 5905 50  0000 L CNN
+F 1 "10k" H 10970 5905 50  0000 L CNN
 F 2 "Resistor_SMD:R_0402_1005Metric" V 10830 5950 50  0001 C CNN
 F 3 "~" H 10900 5950 50  0001 C CNN
+F 4 "RMCF0402FT10K0CT-ND" H 10900 5950 50  0001 C CNN "Digikey"
+F 5 "RMCF0402FT10K0" H 10900 5950 50  0001 C CNN "MPN"
+F 6 "Stackpole" H 10900 5950 50  0001 C CNN "Manufacturer"
 	1    10900 5950
 	1    0    0    -1
@@
 P 8450 5950
 F 0 "R35" H 8520 5996 50  0000 L CNN
-F 1 "10K" H 8520 5905 50  0000 L CNN
+F 1 "10k" H 8520 5905 50  0000 L CNN
 F 2 "Resistor_SMD:R_0402_1005Metric" V 8380 5950 50  0001 C CNN
 F 3 "~" H 8450 5950 50  0001 C CNN
+F 4 "RMCF0402FT10K0CT-ND" H 8450 5950 50  0001 C CNN "Digikey"
+F 5 "RMCF0402FT10K0" H 8450 5950 50  0001 C CNN "MPN"
+F 6 "Stackpole" H 8450 5950 50  0001 C CNN "Manufacturer"
 	1    8450 5950
 	1    0    0    -1
