File: PCB/USB.sch (KiCad schematic (older format))
At the start: 62 parts, among them J5 USB_B, J6 USB_A, J7 To Keyboard, J8 USB_A, J9 USB_A, U6 CY7C65632-28LTXCT, U7 24LC02, U8 MIC2027-2BM, U9 CP2102N-A02-GQFN20, Y2 12MHz

Commit message: WIP PCB changes
Parts:
- removed FL1, FL2, FL3, FL4, FL5: EMI_Filter_CommonMode, symbol Device:EMI_Filter_CommonMode
- removed J7: To Keyboard, symbol Connector_Generic:Conn_01x04
- removed R46, R49, R50, R51: 10K, symbol Device:R
- removed Y2: 12MHz, symbol Device:Crystal_Small
- added D9: DT1240A-08LP3810, Package_DFN_QFN:UDFN-9_1.0x3.8mm_P0.5mm, symbol Power_Protection:DT1240A-08LP3810
- added J5: USB_A, Connector_PinHeader_1.27mm:PinHeader_1x05_P1.27mm_Vertical, symbol Connector:USB_A
- added R64, R65, R66, R67: 10k, Resistor_SMD:R_0402_1005Metric, symbol Device:R
- added Y2: 12MHz, MK_Library:ECS-120-12-36-AGN, symbol Device:Crystal_GND2_Small
- C18: renamed from C24; footprint (none) -> Capacitor_SMD:C_0402_1005Metric; Digikey (none) -> 478-11758-1-ND; MPN (none) -> 04023U200JAT2A; Manufacturer (none) -> AVX
- C19: renamed from C25; footprint (none) -> Capacitor_SMD:C_0402_1005Metric; Digikey (none) -> 478-11758-1-ND; MPN (none) -> 04023U200JAT2A; Manufacturer (none) -> AVX
- C20: renamed from C26; footprint (none) -> Capacitor_SMD:C_0603_1608Metric; Digikey (none) -> 311-4046-1-ND; MPN (none) -> CC0603KRX5R9BB104; Manufacturer (none) -> Yageo
- C21: renamed from C27; footprint (none) -> Capacitor_THT:CP_Radial_D6.3mm_P2.50mm; symbol Device:C_Small -> Device:CP_Small; Digikey (none) -> 732-8511-1-ND; MPN (none) -> 865080545012; Manufacturer (none) -> Würth Elektronik
- C22: renamed from C28; footprint (none) -> Capacitor_SMD:C_0603_1608Metric; Digikey (none) -> 311-4046-1-ND; MPN (none) -> CC0603KRX5R9BB104; Manufacturer (none) -> Yageo
- C23: renamed from C29; footprint (none) -> Capacitor_SMD:C_0603_1608Metric; Digikey (none) -> 311-4046-1-ND; MPN (none) -> CC0603KRX5R9BB104; Manufacturer (none) -> Yageo
- C24: renamed from C30; footprint (none) -> Capacitor_THT:CP_Radial_D6.3mm_P2.50mm; symbol Device:C_Small -> Device:CP_Small; Digikey (none) -> 732-8511-1-ND; MPN (none) -> 865080545012; Manufacturer (none) -> Würth Elektronik
- C25: renamed from C31; footprint (none) -> Capacitor_THT:CP_Radial_D6.3mm_P2.50mm; symbol Device:C_Small -> Device:CP_Small; Digikey (none) -> 732-8511-1-ND; MPN (none) -> 865080545012; Manufacturer (none) -> Würth Elektronik
- C26: renamed from C32; footprint (none) -> Capacitor_SMD:C_0603_1608Metric; Digikey (none) -> 311-4046-1-ND; MPN (none) -> CC0603KRX5R9BB104; Manufacturer (none) -> Yageo
- C27: renamed from C33; footprint (none) -> Capacitor_SMD:C_0603_1608Metric; Digikey (none) -> 311-4046-1-ND; MPN (none) -> CC0603KRX5R9BB104; Manufacturer (none) -> Yageo
- C28: renamed from C34; footprint (none) -> Capacitor_SMD:C_1206_3216Metric; Digikey (none) -> 1276-1055-1-ND; MPN (none) -> CL31B475KAHNNNE; Manufacturer (none) -> Samsung
- C29: renamed from C35; footprint (none) -> Capacitor_SMD:C_0603_1608Metric; Digikey (none) -> 311-4046-1-ND; MPN (none) -> CC0603KRX5R9BB104; Manufacturer (none) -> Yageo
- C30: renamed from C36; footprint (none) -> Capacitor_THT:CP_Radial_D6.3mm_P2.50mm; symbol Device:C_Small -> Device:CP_Small; Digikey (none) -> 732-8511-1-ND; MPN (none) -> 865080545012; Manufacturer (none) -> Würth Elektronik
- C31: renamed from C37; footprint (none) -> Capacitor_THT:CP_Radial_D6.3mm_P2.50mm; symbol Device:C_Small -> Device:CP_Small; Digikey (none) -> 732-8511-1-ND; MPN (none) -> 865080545012; Manufacturer (none) -> Würth Elektronik
- C32: renamed from C38; footprint (none) -> Capacitor_SMD:C_0603_1608Metric; Digikey (none) -> 311-4046-1-ND; MPN (none) -> CC0603KRX5R9BB104; Manufacturer (none) -> Yageo
- C33: renamed from C39; footprint (none) -> Capacitor_SMD:C_0603_1608Metric; Digikey (none) -> 311-4046-1-ND; MPN (none) -> CC0603KRX5R9BB104; Manufacturer (none) -> Yageo
- D10: renamed from D3; footprint (none) -> LED_SMD:LED_0603_1608Metric; Digikey (none) -> 160-1445-1-ND; MPN (none) -> LTST-C191KFKT; Manufacturer (none) -> Lite-On Inc.
- D11: renamed from D4; footprint (none) -> LED_SMD:LED_0603_1608Metric; Digikey (none) -> 160-1445-1-ND; MPN (none) -> LTST-C191KFKT; Manufacturer (none) -> Lite-On Inc.
- D8: renamed from D2; Digikey (none) -> F2715CT-ND; MPN (none) -> SP0503BAHTG; Manufacturer (none) -> Littelfuse Inc.
- FB1, FB10, FB2, FB3, FB4, FB5, FB6, FB7, FB8, FB9: footprint (none) -> Inductor_SMD:L_0805_2012Metric; Digikey (none) -> 490-1054-1-ND; MPN (none) -> BLM21PG221SN1D; Manufacturer (none) -> Murata
- J3: renamed from J5; footprint (none) -> Connector_USB:USB_B_OST_USB-B1HSxx_Horizontal; Digikey (none) -> ED2982-ND; MPN (none) -> USB-B1HSW6; Manufacturer (none) -> On Shore Technology Inc.
- J4: renamed from J6; footprint (none) -> Connector_USB:USB_A_Molex_67643_Horizontal; Digikey (none) -> 2057-USB-A-S-VT-ND; MPN (none) -> USB-A-S-VT; Manufacturer (none) -> Adam Tech
- J6: renamed from J8; footprint (none) -> Connector_PinHeader_1.27mm:PinHeader_1x05_P1.27mm_Vertical; Digikey (none) -> 2057-USB-A-S-VT-ND; MPN (none) -> USB-A-S-VT; Manufacturer (none) -> Adam Tech
- J7: renamed from J9; footprint (none) -> Connector_USB:USB_A_Molex_67643_Horizontal; Digikey (none) -> 2057-USB-A-S-RA-ND; MPN (none) -> USB-A-S-RA; Manufacturer (none) -> Adam Tech
- R10: renamed from R43; footprint (none) -> Resistor_SMD:R_0402_1005Metric; Digikey (none) -> YAG3515CT-ND; MPN (none) -> AC0402JR-07100KL; Manufacturer (none) -> Yageo
- R11: renamed from R44; footprint (none) -> Resistor_SMD:R_0402_1005Metric; Digikey (none) -> P649KLCT-ND; MPN (none) -> ERJ-2RKF6493X; Manufacturer (none) -> Panasonic Electronic Components
- R12: renamed from R45; footprint (none) -> Resistor_SMD:R_0402_1005Metric; Digikey (none) -> RMCF0402FT10K0CT-ND; MPN (none) -> RMCF0402FT10K0; Manufacturer (none) -> Stackpole
- R13: renamed from R47; footprint (none) -> Resistor_SMD:R_0402_1005Metric; Digikey (none) -> RMCF0402FT10K0CT-ND; MPN (none) -> RMCF0402FT10K0; Manufacturer (none) -> Stackpole
- R14: renamed from R48; footprint (none) -> Resistor_SMD:R_0402_1005Metric
- R15: renamed from R52; footprint (none) -> Resistor_SMD:R_0402_1005Metric; Digikey (none) -> YAG3457CT-ND; MPN (none) -> AC0402FR-0722K1L; Manufacturer (none) -> Yageo
- R16: renamed from R53; footprint (none) -> Resistor_SMD:R_0402_1005Metric; Digikey (none) -> RMCF0402FT47K5CT-ND; MPN (none) -> RMCF0402FT47K5; Manufacturer (none) -> Stackpole
- R17: renamed from R54; value 1k -> 10k; footprint (none) -> Resistor_SMD:R_0402_1005Metric; Digikey (none) -> RMCF0402FT10K0CT-ND; MPN (none) -> RMCF0402FT10K0; Manufacturer (none) -> Stackpole
- R18: renamed from R55; value 390R -> 270R; footprint (none) -> Resistor_SMD:R_0402_1005Metric; Digikey (none) -> 311-270JRCT-ND; MPN (none) -> RC0402JR-07270RL; Manufacturer (none) -> Yageo
- R19: renamed from R56; value 390R -> 270R; footprint (none) -> Resistor_SMD:R_0402_1005Metric; Digikey (none) -> 311-270JRCT-ND; MPN (none) -> RC0402JR-07270RL; Manufacturer (none) -> Yageo
- R20: renamed from R57; footprint (none) -> Resistor_SMD:R_0402_1005Metric; Digikey (none) -> RMCF0402FT10K0CT-ND; MPN (none) -> RMCF0402FT10K0; Manufacturer (none) -> Stackpole
- R9: renamed from R42; footprint (none) -> Resistor_SMD:R_0402_1005Metric; Digikey (none) -> RMCF0402FT10K0CT-ND; MPN (none) -> RMCF0402FT10K0; Manufacturer (none) -> Stackpole
- TP2, TP3: footprint (none) -> TestPoint:TestPoint_Pad_1.5x1.5mm
- U3: renamed from U6; value CY7C65632-28LTXCT -> CY7C65632-28LTXC; footprint QFN-28 -> Package_DFN_QFN:QFN-28-1EP_5x5mm_P0.5mm_EP3.35x3.35mm; Digikey (none) -> CY7C65632-28LTXC-ND; MPN (none) -> CY7C65632-28LTXC; Manufacturer (none) -> Cypress Semiconductor
- U4: renamed from U7; footprint (none) -> Package_SO:SOIC-8_3.9x4.9mm_P1.27mm; Digikey (none) -> 24LC02BT/SN; MPN (none) -> 24LC02BT/SNCT-ND; Manufacturer (none) -> Microchip
- U5: renamed from U8; footprint Housings_SOIC:SOIC-16_3.9x9.9mm_Pitch1.27mm -> Package_SO:SOIC-16_3.9x9.9mm_P1.27mm; Digikey (none) -> 576-2138-ND; MPN (none) -> MIC2027-1YM; Manufacturer (none) -> Microchip Technology
- U6: renamed from U9; footprint (none) -> Package_DFN_QFN:QFN-24-1EP_4x4mm_P0.5mm_EP2.6x2.6mm; Digikey (none) -> 336-5885-ND; MPN (none) -> CP2102N-A02; Mouser (none) -> 634-CP2102NA02QFN20R
Connections:
- net D_MLC_N is gone; now on net D1N: U6.5 (D-)
- net D_MLC_P is gone; now on net D1P: U6.4 (D+)
- net +3V3: now also R64.1, R65.1, R66.1, R67.1
- net D2N: now also J5.2 (D-)
- net D2P: now also J5.3 (D+)
- net D3N: now also J6.2 (D-), D9.9 (K8)
- net D3P: now also J6.3 (D+), D9.8 (K7)
- net D4N: now also J7.2 (D-), D9.7 (K6)
- net D4P: now also J7.3 (D+), D9.6 (K5)
- net DIN_N: now also J3.2 (D-)
- net DIN_P: now also J3.3 (D+)
- net GND: now also D9.3 (A), Y2.2; no longer C21.2, C26.2, C27.2, C32.2, C33.2, FB10.1, FB2.2, FB4.1, FB6.1, FB8.1, J3.4 (GND), J4.4 (GND), J4.5 (Shield), J6.4 (GND), J6.5 (Shield), J7.4 (GND), J7.5 (Shield)
- net VBUS_C: now also C30.1, FB7.2; no longer C31.1, FB9.2
- net VBUS_D: now also C31.1, FB9.2; no longer C30.1, FB7.2
- net XIN: now also Y2.1
- net XOUT: now also Y2.3
- net ~OVR1: now reaches U3.25 (~OVR1), U5.1 (FLGA)
- net ~OVR1: now also R64.2
- net ~OVR2: now reaches U3.24 (~OVR2), U5.16 (FLGB)
- net ~OVR2: now also R65.2
- net ~OVR3: now reaches U3.20 (~OVR3), U5.8 (FLGC)
- net ~OVR3: now also R66.2
- net ~OVR4: now reaches U3.19 (~OVR4), U5.9 (FLGD)
- net ~OVR4: now also R67.2
- net at C26.1, FB3.1: now also J5.1 (VBUS)
- net at R9.2, U3.17 (~RESET): no longer U3.22 (SELFPWR)
- new net: C26.2, FB4.1, J5.4 (GND), J5.5 (Shield)
- new net: C32.2, FB8.1, J6.4 (GND), J6.5 (Shield)
- new net: C33.2, FB10.1, J7.4 (GND), J7.5 (Shield)
- new net: C21.2, FB2.2, J3.4 (GND)
- new net: C27.2, FB6.1, J4.4 (GND), J4.5 (Shield)
- new net SELF_POWER: U3.22 (SELFPWR)
Other:
- note added: "ESD Protection"
- note added: "Hardwired Connection\n(Internal)"
- note added: "To Keyboard\n(Internal)"
- note added: "To Panel USB"
- note added: "To Rear USB\n(Power + Data)"
- note added: "USB Controller, Bus Voltage Controller"
- note removed: "To Panel USB 1"
- note removed: "To Panel USB 2"
- note removed: "USB and Bus Voltage Controller"

Commit message: PCB Version 1: As Sent to Fab
Parts:
- added R32: 10k, Resistor_SMD:R_0402_1005Metric, symbol Device:R
- C20, C22, C23, C26, C27, C29, C32, C33: Digikey 311-4046-1-ND -> 587-1243-1-ND; MPN CC0603KRX5R9BB104 -> UMK107B7104KA-T; Manufacturer Yageo -> Taiyo Yuden
- D10, D11: value LED -> LED_Orange
- D9: Digikey (none) -> DT1240A-08LP3810-7DICT-ND
- J4: Digikey 2057-USB-A-S-VT-ND -> WM14667-ND; MPN USB-A-S-VT -> 0676433910; Manufacturer Adam Tech -> Molex
- J5, J6: Digikey 2057-USB-A-S-VT-ND -> (none)
- J7: Digikey 2057-USB-A-S-RA-ND -> WM14667-ND; MPN USB-A-S-RA -> 0676433910; Manufacturer Adam Tech -> Molex
- R10: Digikey YAG3515CT-ND -> RMCF0402FT100KCT-ND
- R64, R65, R66, R67: Digikey (none) -> RMCF0402FT10K0CT-ND; MPN (none) -> RMCF0402FT10K0; Manufacturer (none) -> Stackpole
Connections:
- net GND: now also R32.1; no longer R14.2, U4.7 (WP)
- new net: R14.2, R32.2, U4.7 (WP)
Changed lines of the file:
@@
 F 2 "Capacitor_SMD:C_0603_1608Metric" H 12100 1950 50  0001 C CNN
 F 3 "~" H 12100 1950 50  0001 C CNN
-F 4 "311-4046-1-ND" H 12100 1950 50  0001 C CNN "Digikey"
-F 5 "CC0603KRX5R9BB104" H 12100 1950 50  0001 C CNN "MPN"
-F 6 "Yageo" H 12100 1950 50  0001 C CNN "Manufacturer"
+F 4 "587-1243-1-ND" H 12100 1950 50  0001 C CNN "Digikey"
+F 5 "UMK107B7104KA-T" H 12100 1950 50  0001 C CNN "MPN"
+F 6 "Taiyo Yuden" H 12100 1950 50  0001 C CNN "Manufacturer"
 	1    12100 1950
 	0    1    1    0
@@
 F 2 "Connector_PinHeader_1.27mm:PinHeader_1x05_P1.27mm_Vertical" H 15200 7000 50  0001 C CNN
 F 3 " ~" H 15200 7000 50  0001 C CNN
-F 4 "2057-USB-A-S-VT-ND" H 15050 7050 50  0001 C CNN "Digikey"
+F 4 "" H 15050 7050 50  0001 C CNN "Digikey"
 F 5 "USB-A-S-VT" H 15050 7050 50  0001 C CNN "MPN"
 F 6 "Adam Tech" H 15050 7050 50  0001 C CNN "Manufacturer"
@@
 F 2 "Capacitor_SMD:C_0603_1608Metric" H 13300 7100 50  0001 C CNN
 F 3 "~" H 13300 7100 50  0001 C CNN
-F 4 "311-4046-1-ND" H 13300 7100 50  0001 C CNN "Digikey"
-F 5 "CC0603KRX5R9BB104" H 13300 7100 50  0001 C CNN "MPN"
-F 6 "Yageo" H 13300 7100 50  0001 C CNN "Manufacturer"
+F 4 "587-1243-1-ND" H 13300 7100 50  0001 C CNN "Digikey"
+F 5 "UMK107B7104KA-T" H 13300 7100 50  0001 C CNN "MPN"
+F 6 "Taiyo Yuden" H 13300 7100 50  0001 C CNN "Manufacturer"
 	1    13300 7100
 	1    0    0    -1
@@
 F 2 "Connector_USB:USB_A_Molex_67643_Horizontal" H 15250 5750 50  0001 C CNN
 F 3 " ~" H 15250 5750 50  0001 C CNN
-F 4 "2057-USB-A-S-RA-ND" H 15100 5800 50  0001 C CNN "Digikey"
-F 5 "USB-A-S-RA" H 15100 5800 50  0001 C CNN "MPN"
-F 6 "Adam Tech" H 15100 5800 50  0001 C CNN "Manufacturer"
+F 4 "WM14667-ND" H 15100 5800 50  0001 C CNN "Digikey"
+F 5 "0676433910" H 15100 5800 50  0001 C CNN "MPN"
+F 6 "Molex" H 15100 5800 50  0001 C CNN "Manufacturer"
 	1    15100 5800
 	-1   0    0    -1
@@
 F 2 "Capacitor_SMD:C_0603_1608Metric" H 13350 5850 50  0001 C CNN
 F 3 "~" H 13350 5850 50  0001 C CNN
-F 4 "311-4046-1-ND" H 13350 5850 50  0001 C CNN "Digikey"
-F 5 "CC0603KRX5R9BB104" H 13350 5850 50  0001 C CNN "MPN"
-F 6 "Yageo" H 13350 5850 50  0001 C CNN "Manufacturer"
+F 4 "587-1243-1-ND" H 13350 5850 50  0001 C CNN "Digikey"
+F 5 "UMK107B7104KA-T" H 13350 5850 50  0001 C CNN "MPN"
+F 6 "Taiyo Yuden" H 13350 5850 50  0001 C CNN "Manufacturer"
 	1    13350 5850
 	1    0    0    -1
@@
 F 2 "Capacitor_SMD:C_0603_1608Metric" H 10100 7100 50  0001 C CNN
 F 3 "~" H 10100 7100 50  0001 C CNN
-F 4 "311-4046-1-ND" H 10100 7100 50  0001 C CNN "Digikey"
-F 5 "CC0603KRX5R9BB104" H 10100 7100 50  0001 C CNN "MPN"
-F 6 "Yageo" H 10100 7100 50  0001 C CNN "Manufacturer"
+F 4 "587-1243-1-ND" H 10100 7100 50  0001 C CNN "Digikey"
+F 5 "UMK107B7104KA-T" H 10100 7100 50  0001 C CNN "MPN"
+F 6 "Taiyo Yuden" H 10100 7100 50  0001 C CNN "Manufacturer"
 	1    10100 7100
 	1    0    0    -1
@@
 F 2 "Capacitor_SMD:C_0603_1608Metric" H 6150 5350 50  0001 C CNN
 F 3 "~" H 6150 5350 50  0001 C CNN
-F 4 "311-4046-1-ND" H 6150 5350 50  0001 C CNN "Digikey"
-F 5 "CC0603KRX5R9BB104" H 6150 5350 50  0001 C CNN "MPN"
-F 6 "Yageo" H 6150 5350 50  0001 C CNN "Manufacturer"
+F 4 "587-1243-1-ND" H 6150 5350 50  0001 C CNN "Digikey"
+F 5 "UMK107B7104KA-T" H 6150 5350 50  0001 C CNN "MPN"
+F 6 "Taiyo Yuden" H 6150 5350 50  0001 C CNN "Manufacturer"
 	1    6150 5350
 	-1   0    0    1
@@
 F 2 "Capacitor_SMD:C_0603_1608Metric" H 5450 2250 50  0001 C CNN
 F 3 "~" H 5450 2250 50  0001 C CNN
-F 4 "311-4046-1-ND" H 5450 2250 50  0001 C CNN "Digikey"
-F 5 "CC0603KRX5R9BB104" H 5450 2250 50  0001 C CNN "MPN"
-F 6 "Yageo" H 5450 2250 50  0001 C CNN "Manufacturer"
+F 4 "587-1243-1-ND" H 5450 2250 50  0001 C CNN "Digikey"
+F 5 "UMK107B7104KA-T" H 5450 2250 50  0001 C CNN "MPN"
+F 6 "Taiyo Yuden" H 5450 2250 50  0001 C CNN "Manufacturer"
 	1    5450 2250
 	1    0    0    -1
@@
 F 2 "Resistor_SMD:R_0402_1005Metric" V 1930 5850 50  0001 C CNN
 F 3 "~" H 2000 5850 50  0001 C CNN
-F 4 "YAG3515CT-ND" H 2000 5850 50  0001 C CNN "Digikey"
+F 4 "RMCF0402FT100KCT-ND" H 2000 5850 50  0001 C CNN "Digikey"
 F 5 "AC0402JR-07100KL" H 2000 5850 50  0001 C CNN "MPN"
 F 6 "Yageo" H 2000 5850 50  0001 C CNN "Manufacturer"
@@
 	4300 9000 4300 9050
 Wire Wire Line
-	4700 8800 4800 8800
-Wire Wire Line
-	4800 8800 4800 9050
-Wire Wire Line
 	4700 8700 5050 8700
 Wire Wire Line
@@
 L power:GND #PWR070
 U 1 1 5FDB86C2
-P 4800 9050
-F 0 "#PWR070" H 4800 8800 50  0001 C CNN
-F 1 "GND" H 4805 8877 50  0000 C CNN
-F 2 "" H 4800 9050 50  0001 C CNN
-F 3 "" H 4800 9050 50  0001 C CNN
-	1    4800 9050
+P 4800 9150
+F 0 "#PWR070" H 4800 8900 50  0001 C CNN
+F 1 "GND" H 4805 8977 50  0000 C CNN
+F 2 "" H 4800 9150 50  0001 C CNN
+F 3 "" H 4800 9150 50  0001 C CNN
+	1    4800 9150
 	1    0    0    -1
 $EndComp
@@
 	0    1    1    0
 $EndComp
-Wire Wire Line
-	4900 8800 4800 8800
-Connection ~ 4800 8800
 Wire Wire Line
 	5200 8800 5850 8800
@@
 F 2 "Capacitor_SMD:C_0603_1608Metric" H 4150 8100 50  0001 C CNN
 F 3 "~" H 4150 8100 50  0001 C CNN
-F 4 "311-4046-1-ND" H 4150 8100 50  0001 C CNN "Digikey"
-F 5 "CC0603KRX5R9BB104" H 4150 8100 50  0001 C CNN "MPN"
-F 6 "Yageo" H 4150 8100 50  0001 C CNN "Manufacturer"
+F 4 "587-1243-1-ND" H 4150 8100 50  0001 C CNN "Digikey"
+F 5 "UMK107B7104KA-T" H 4150 8100 50  0001 C CNN "MPN"
+F 6 "Taiyo Yuden" H 4150 8100 50  0001 C CNN "Manufacturer"
 	1    4150 8100
 	-1   0    0    1
@@
 P 13650 3150
 F 0 "D10" V 13700 3350 50  0000 R CNN
-F 1 "LED" V 13600 3350 50  0000 R CNN
+F 1 "LED_Orange" V 13600 3350 50  0000 R CNN
 F 2 "LED_SMD:LED_0603_1608Metric" H 13650 3150 50  0001 C CNN
 F 3 "~" H 13650 3150 50  0001 C CNN
@@
 P 13900 3150
 F 0 "D11" V 13939 3033 50  0000 R CNN
-F 1 "LED" V 13848 3033 50  0000 R CNN
+F 1 "LED_Orange" V 13848 3033 50  0000 R CNN
 F 2 "LED_SMD:LED_0603_1608Metric" H 13900 3150 50  0001 C CNN
 F 3 "~" H 13900 3150 50  0001 C CNN
@@
 AR Path="/60B6F3FC" Ref="J?"  Part="1"
 AR Path="/5FF26B81/60B6F3FC" Ref="J4"  Part="1"
+AR Path="/5F4A9D3D/60B6F3FC" Ref="J4"  Part="1"
 F 0 "J4" H 10620 5789 50  0000 R CNN
 F 1 "USB_A" H 10620 5698 50  0000 R CNN
 F 2 "Connector_USB:USB_A_Molex_67643_Horizontal" H 11000 5750 50  0001 C CNN
 F 3 " ~" H 11000 5750 50  0001 C CNN
-F 4 "2057-USB-A-S-VT-ND" H 10850 5800 50  0001 C CNN "Digikey"
-F 5 "USB-A-S-VT" H 10850 5800 50  0001 C CNN "MPN"
-F 6 "Adam Tech" H 10850 5800 50  0001 C CNN "Manufacturer"
+F 4 "WM14667-ND" H 10850 5800 50  0001 C CNN "Digikey"
+F 5 "0676433910" H 10850 5800 50  0001 C CNN "MPN"
+F 6 "Molex" H 10850 5800 50  0001 C CNN "Manufacturer"
 	1    10850 5800
 	-1   0    0    -1
@@
 F 2 "Capacitor_SMD:C_0603_1608Metric" H 10150 5850 50  0001 C CNN
 F 3 "~" H 10150 5850 50  0001 C CNN
-F 4 "311-4046-1-ND" H 10150 5850 50  0001 C CNN "Digikey"
-F 5 "CC0603KRX5R9BB104" H 10150 5850 50  0001 C CNN "MPN"
-F 6 "Yageo" H 10150 5850 50  0001 C CNN "Manufacturer"
+F 4 "587-1243-1-ND" H 10150 5850 50  0001 C CNN "Digikey"
+F 5 "UMK107B7104KA-T" H 10150 5850 50  0001 C CNN "MPN"
+F 6 "Taiyo Yuden" H 10150 5850 50  0001 C CNN "Manufacturer"
 	1    10150 5850
 	1    0    0    -1
@@
 F 2 "Connector_PinHeader_1.27mm:PinHeader_1x05_P1.27mm_Vertical" H 11850 7000 50  0001 C CNN
 F 3 " ~" H 11850 7000 50  0001 C CNN
-F 4 "2057-USB-A-S-VT-ND" H 11700 7050 50  0001 C CNN "Digikey"
+F 4 "" H 11700 7050 50  0001 C CNN "Digikey"
 F 5 "USB-A-S-VT" H 11700 7050 50  0001 C CNN "MPN"
 F 6 "Adam Tech" H 11700 7050 50  0001 C CNN "Manufacturer"
@@
 F 2 "Package_DFN_QFN:UDFN-9_1.0x3.8mm_P0.5mm" H 10350 8850 50  0001 L CNN
 F 3 "https://www.diodes.com/assets/Datasheets/DT1240A-08LP3810.pdf" H 9975 8925 50  0001 C CNN
+F 4 "DT1240A-08LP3810-7DICT-ND" H 9800 8900 50  0001 C CNN "Digikey"
 	1    9800 8900
 	0    1    1    0
@@
 F 2 "Resistor_SMD:R_0402_1005Metric" V 4830 5350 50  0001 C CNN
 F 3 "~" H 4900 5350 50  0001 C CNN
+F 4 "RMCF0402FT10K0CT-ND" H 4900 5350 50  0001 C CNN "Digikey"
+F 5 "RMCF0402FT10K0" H 4900 5350 50  0001 C CNN "MPN"
+F 6 "Stackpole" H 4900 5350 50  0001 C CNN "Manufacturer"
 	1    4900 5350
 	1    0    0    -1
@@
 F 2 "Resistor_SMD:R_0402_1005Metric" V 5130 5350 50  0001 C CNN
 F 3 "~" H 5200 5350 50  0001 C CNN
+F 4 "RMCF0402FT10K0CT-ND" H 5200 5350 50  0001 C CNN "Digikey"
+F 5 "RMCF0402FT10K0" H 5200 5350 50  0001 C CNN "MPN"
+F 6 "Stackpole" H 5200 5350 50  0001 C CNN "Manufacturer"
 	1    5200 5350
 	1    0    0    -1
@@
 F 2 "Resistor_SMD:R_0402_1005Metric" V 5430 5350 50  0001 C CNN
 F 3 "~" H 5500 5350 50  0001 C CNN
+F 4 "RMCF0402FT10K0CT-ND" H 5500 5350 50  0001 C CNN "Digikey"
+F 5 "RMCF0402FT10K0" H 5500 5350 50  0001 C CNN "MPN"
+F 6 "Stackpole" H 5500 5350 50  0001 C CNN "Manufacturer"
 	1    5500 5350
 	1    0    0    -1
@@
 F 2 "Resistor_SMD:R_0402_1005Metric" V 5730 5350 50  0001 C CNN
 F 3 "~" H 5800 5350 50  0001 C CNN
+F 4 "RMCF0402FT10K0CT-ND" H 5800 5350 50  0001 C CNN "Digikey"
+F 5 "RMCF0402FT10K0" H 5800 5350 50  0001 C CNN "MPN"
+F 6 "Stackpole" H 5800 5350 50  0001 C CNN "Manufacturer"
 	1    5800 5350
 	1    0    0    -1
@@
 Text Label 4350 6600 2    50   ~ 0
 ~OVR4
+Wire Wire Line
+	4700 8800 4800 8800
+$Comp
+L Device:R R32
+U 1 1 5FB5FE6E
+P 4800 8950
+F 0 "R32" V 4900 8950 50  0000 C CNN
+F 1 "10k" V 4800 8950 50  0000 C CNN
+F 2 "Resistor_SMD:R_0402_1005Metric" V 4730 8950 50  0001 C CNN
+F 3 "~" H 4800 8950 50  0001 C CNN
+F 4 "RMCF0402FT10K0CT-ND" H 4800 8950 50  0001 C CNN "Digikey"
+F 5 "RMCF0402FT10K0" H 4800 8950 50  0001 C CNN "MPN"
+F 6 "Stackpole" H 4800 8950 50  0001 C CNN "Manufacturer"
+	1    4800 8950
+	-1   0    0    1
+$EndComp
+Connection ~ 4800 8800
+Wire Wire Line
+	4800 8800 4900 8800
+Wire Wire Line
+	4800 9100 4800 9150
 $EndSCHEMATC
