File: PCB/V2/Console.kicad_pcb (KiCad board)
At the start: 2 copper layers, 168 x 72.5 mm, 191 parts, among them J1 SliderConnector, J10 EncoderConnector, J11 EncoderConnector, J12 EncoderConnector, J13 EncoderConnector, J2 SliderConnector, J3 USB_B, J4 USB_A, J5 USB_A, J6 USB_A, J7 USB_A, J8 Barrel_Jack_Switch, J9 SliderConnector, Q1 FDN338P, Q2 MMBT3904, Q3 FDN338P, SW1 SW_Push_LED, SW10 Rotary_Encoder_Switch, SW11 SW_Push, SW12 SW_Push, SW2 SW_Push_LED, SW3 SW_Push_LED, SW4 SW_Push_LED, SW5 SW_Push_LED, SW6 SW_Push_LED, SW7 Rotary_Encoder_Switch, SW8 Rotary_Encoder_Switch, SW9 Rotary_Encoder_Switch, U1 CP2102N-A01-GQFN28, U10 NHD-3.12-25664UCW2, U2 MCP23017_SO, U3 CY7C65632-28LTXC, U4 24LC02, U5 MIC2027, U7 DMP1005UFDF, U8 AP2114HA-3.3TRG1, U9 ESP32-WROOM-32, Y2 12MHz

Commit message: PCB Sent
Parts:
- added C29: 4.7uF, Capacitor_SMD:C_0805_2012Metric, B.Cu at (161.2, 109.5)
- added C44: 0.1uF, Capacitor_SMD:C_0402_1005Metric, B.Cu at (160.5, 108.0)
- added TP10: TestPoint, TestPoint:TestPoint_Pad_1.5x1.5mm, B.Cu at (126.2, 118.5)
- added TP7: TestPoint, TestPoint:TestPoint_Pad_1.5x1.5mm, F.Cu at (110.2, 123.2)
- added TP8: TestPoint, TestPoint:TestPoint_Pad_1.5x1.5mm, B.Cu at (119.0, 118.5)
- added TP9: TestPoint, TestPoint:TestPoint_Pad_1.5x1.5mm, B.Cu at (116.2, 118.5)
- added U6: CP2110-24QFN, Package_DFN_QFN:QFN-24-1EP_4x4mm_P0.5mm_EP2.7x2.7mm, B.Cu at (156.8, 107.0)
- C1, C2, C35, C36, C38, C42, C5: footprint Capacitor_SMD:C_1206_3216Metric -> Capacitor_SMD:C_0805_2012Metric
- J1, J2, J9: footprint Connector_JST:JST_EH_B3B-EH-A_1x03_P2.50mm_Vertical -> Connector_JST:JST_PH_S3B-PH-K_1x03_P2.00mm_Horizontal
- Q1, Q3: value FDN338P -> CPH3356-TL-W
- TP4: moved to B.Cu
- U10: value NHD-3.12-25664UCW2 -> 1-535541-8 (Connector)
- moved H10 70.5 mm to (158.2, 97.0)
- moved R2 69.4 mm to (225.6, 87.4), turned to 90 degrees
- moved Q3 63.7 mm to (219.4, 88.2), turned to 0 degrees
- moved Q2 62.8 mm to (223.2, 88.2), turned to 270 degrees
- moved R15 59.7 mm to (216.4, 89.2), turned to 270 degrees
- moved R36 41.7 mm to (171.4, 109.4), turned to 180 degrees
- moved R39 39.3 mm to (171.4, 111.5), turned to 180 degrees
- moved FB8 29.5 mm to (219.6, 63.4), turned to 270 degrees
- moved C32 27.8 mm to (212.9, 60.2), turned to 0 degrees
- moved C30 23.9 mm to (215.6, 65.2), turned to 0 degrees
- moved R35 23.8 mm to (171.4, 107.8), turned to 180 degrees
- moved J6 22.6 mm to (212.4, 62.4), turned to 90 degrees
- moved FB7 20.9 mm to (212.5, 65.2)
- moved R38 20.2 mm to (171.4, 113.1), turned to 180 degrees
- moved FB6 18.1 mm to (215.2, 71.5), turned to 90 degrees
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Connections:
- net Net-(C2-Pad2) renamed /Core/VPP
- net Net-(R20-Pad1) renamed /Core/RSTb
- J1 pad 1: +3V3 -> /Core/SLD1
- J1 pad 2: /Core/SLD1 -> +3V3
- J2 pad 1: +3V3 -> /Core/SLD2
- J2 pad 2: /Core/SLD2 -> +3V3
- J9 pad 1: +3V3 -> /Core/SLD3
- J9 pad 2: /Core/SLD3 -> +3V3
- R3 pad 1: LED_Power -> Net-(R3-Pad1)
- R3 pad 2: Net-(R3-Pad2) -> GND
- R4 pad 1: LED_Power -> Net-(R4-Pad1)
- R4 pad 2: Net-(R4-Pad2) -> GND
- R5 pad 1: LED_Power -> Net-(R5-Pad1)
- R5 pad 2: Net-(R5-Pad2) -> GND
- R6 pad 1: LED_Power -> Net-(R6-Pad1)
- R6 pad 2: Net-(R6-Pad2) -> GND
- R7 pad 1: LED_Power -> Net-(R7-Pad1)
- R7 pad 2: Net-(R7-Pad2) -> GND
- R74 pad 1: /Core/OLED_~RESET -> /Core/OLED_~CS
- R8 pad 1: LED_Power -> Net-(R8-Pad1)
- R8 pad 2: Net-(R8-Pad2) -> GND
- SW1 pad 3: GND -> Net-(R3-Pad1)
- SW1 pad 4: Net-(R3-Pad2) -> LED_Power
- SW2 pad 3: GND -> Net-(R4-Pad1)
- SW2 pad 4: Net-(R4-Pad2) -> LED_Power
- SW3 pad 3: GND -> Net-(R5-Pad1)
- SW3 pad 4: Net-(R5-Pad2) -> LED_Power
- SW4 pad 3: GND -> Net-(R6-Pad1)
- SW4 pad 4: Net-(R6-Pad2) -> LED_Power
- SW5 pad 3: GND -> Net-(R7-Pad1)
- SW5 pad 4: Net-(R7-Pad2) -> LED_Power
- SW6 pad 3: GND -> Net-(R8-Pad1)
- SW6 pad 4: Net-(R8-Pad2) -> LED_Power
- TP4 pad 1: /Core/SPARE1 -> /Core/SPARE4
- U9 pad 10: /Core/ENC2_A -> /Core/ENC2_B
- U9 pad 13: Net-(TP9-Pad1) -> /Core/SPARE2
- U9 pad 23: Net-(TP10-Pad1) -> /Core/SPARE3
- U9 pad 24: /Core/OLED_~CS -> /Core/OLED_~RESET
- U9 pad 27: /Core/ENC4_B -> /Core/ENC4_A
- U9 pad 28: /Core/ENC4_A -> /Core/ENC4_B
- U9 pad 31: /Core/SPARE1 -> /Core/SPARE4
- U9 pad 9: /Core/ENC2_B -> /Core/ENC2_A
Routing:
- net +3V3: track 343.0 -> 626.8 mm, vias 17 -> 34
- net /Core/LED_PWM: track 0.00 -> 144.2 mm, vias 0 -> 4
- net /Peripherals/ENC1_SW: track 0.00 -> 88.4 mm, vias 0 -> 2
- net /USB Hub and Serial Converter/USB_INT_P: track 0.00 -> 72.4 mm, vias 0 -> 2
- net /USB Hub and Serial Converter/USB_INT_N: track 0.00 -> 69.5 mm, vias 0 -> 2
- net /Peripherals/ENC2_SW: track 0.00 -> 68.6 mm, vias 0 -> 2
- net /USB Hub and Serial Converter/D3P: track 4.38 -> 65.0 mm, vias 0 -> 3
- net /USB Hub and Serial Converter/D3N: track 5.37 -> 65.1 mm, vias 0 -> 3
- net /Core/EN: track 0.00 -> 57.7 mm, vias 0 -> 2
- net /Core/SLD1: track 0.00 -> 56.5 mm, vias 0 -> 1
- net /Power/SELF_POWER: track 9.07 -> 64.1 mm, vias 1 -> 2
- net /Core/ENC1_B: track 0.00 -> 53.7 mm, vias 0 -> 2
- net /Core/ENC1_A: track 0.00 -> 52.4 mm, vias 0 -> 2
- net /Core/ENC3_A: track 0.00 -> 52.1 mm, vias 0 -> 2
- net /Core/ENC3_B: track 0.00 -> 49.9 mm, vias 0 -> 2
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