File: PCB/V2/Core.sch (KiCad schematic (older format))
At the start: 41 parts, among them SW11 SW_Push, SW12 SW_Push, U1 CP2102N-A01-GQFN28, U10 NHD-3.12-25664UCW2, U9 ESP32-WROOM-32

Commit message: PCB Sent
Parts:
- added ANT1: Antenna, symbol Graphic:SYM_Arrow_Normal
- added C29: 4.7uF, Capacitor_SMD:C_0805_2012Metric, symbol Device:C_Small
- added C44: 0.1uF, Capacitor_SMD:C_0402_1005Metric, symbol Device:C_Small
- added CON1: AntennaConnector, symbol Graphic:SYM_Arrow_Normal
- added OLED1: Newhaven OLED, symbol Graphic:SYM_Arrow_Normal
- added U6: CP2110-24QFN, Package_DFN_QFN:QFN-24-1EP_4x4mm_P0.5mm_EP2.7x2.7mm, symbol MK_Library:CP2110-24QFN
- C1, C2, C42: footprint Capacitor_SMD:C_1206_3216Metric -> Capacitor_SMD:C_0805_2012Metric; Digikey 1276-1055-1-ND -> 1276-1244-1-ND
- C39: Digikey 1276-6687-1-ND -> 1276-2909-1-ND
- D17: Digikey 160-1446-1-ND -> 160-1183-1-ND
- U10: value NHD-3.12-25664UCW2 -> 1-535541-8 (Connector); Digikey NHD-3.12-25664UCW2-ND -> A26483-ND; MPN NHD-3.12-25664UCW2 -> (none); Manufacturer Newhaven Display Intl -> (none)
- U9: Digikey 1904-1028-1-ND -> 1965-ESP32-WROOM-32UE(4MB)CT-ND
Connections:
- net +3V3: now also C29.2, C44.2, U6.5 (VIO), U6.6 (VDD), U6.7 (REGIN)
- net ENC2_A: now also U9.9 (IO33); no longer U9.10 (IO25)
- net ENC2_B: now also U9.10 (IO25); no longer U9.9 (IO33)
- net ENC4_A: now also U9.27 (IO16); no longer U9.28 (IO17)
- net ENC4_B: now also U9.28 (IO17); no longer U9.27 (IO16)
- net GND: now also C29.1, C44.1, U6.2 (GND), U6.25 (GND)
- net OLED_~CS: now also R74.1; no longer U9.24 (IO2)
- net OLED_~RESET: now also U9.24 (IO2); no longer R74.1
- net RXD0: now also U6.20 (RX)
- net RXT: now also U6.18 (RXT/GPIO.5)
- net SPARE1: no longer TP4.1, U9.31 (IO19)
- net SUS_SENSE: now also U6.11 (SUSPEND)
- net TXD0: now also U6.21 (TX)
- net TXT: now also U6.19 (TXT/GPIO.4)
- net USB_N: now also U6.4 (D-)
- net USB_P: now also U6.3 (D+)
- net VBUS_SENSE: now also U6.8 (VBUS)
- net SPARE2: now reaches TP9.1, U9.13 (IO14)
- net SPARE3: now reaches TP10.1, U9.23 (IO15)
- net VPP: now reaches C2.2, R68.2, U1.18 (~RXT~/GPIO.1)
- net VPP: now also U6.16 (VPP)
- net RSTb: now reaches R20.1, U1.9 (~RSTb)
- net RSTb: now also U6.9 (~RST)
- new net SPARE4: TP4.1, U9.31 (IO19)
- no-connect marks 20 -> 29
Other:
- note added: "Spare Footprint for 24QFN CP2110"
- moved on the sheet: R20
