File: PCB/V2/EncoderCircuit.sch (KiCad schematic (older format))
At the start: 12 parts, among them J12 EncoderConnector, SW7 Rotary_Encoder_Switch

Commit message: PCB Sent
Parts:
- J12: Digikey 455-1752-1-ND -> 455-1722-ND
Changed lines of the file:
@@
 $Descr USLetter 11000 8500
 encoding utf-8
-Sheet 4 9
+Sheet 6 9
 Title "EMRSNxEOS Console"
 Date ""
@@
 AR Path="/5F4A9E86/5F6DDF02/5F69EEA5" Ref="SW10"  Part="1"
 AR Path="/5F4A9E86/5F60074F/5F69EEA5" Ref="SW?"  Part="1"
-F 0 "SW8" H 5950 4050 50  0000 C CNN
+F 0 "SW10" H 5950 4050 50  0000 C CNN
 F 1 "Rotary_Encoder_Switch" H 5750 3550 50  0000 C CNN
 F 2 "MK_Library:BOM_ONLY" H 5800 3960 50  0001 C CNN
@@
 AR Path="/5F4A9E86/5F6DDF02/5F6B8BDC" Ref="C15"  Part="1"
 AR Path="/5F4A9E86/5F60074F/5F6B8BDC" Ref="C?"  Part="1"
-F 0 "C9" H 3550 4050 50  0000 L CNN
+F 0 "C15" H 3550 4050 50  0000 L CNN
 F 1 "10n" H 3550 3950 50  0000 L CNN
 F 2 "Capacitor_SMD:C_0402_1005Metric" H 3838 3950 50  0001 C CNN
@@
 AR Path="/5F4A9E86/5F6DDF02/5F6B95E0" Ref="C16"  Part="1"
 AR Path="/5F4A9E86/5F60074F/5F6B95E0" Ref="C?"  Part="1"
-F 0 "C10" H 4250 4050 50  0000 L CNN
+F 0 "C16" H 4250 4050 50  0000 L CNN
 F 1 "10n" H 4250 3950 50  0000 L CNN
 F 2 "Capacitor_SMD:C_0402_1005Metric" H 4188 3950 50  0001 C CNN
@@
 AR Path="/5F4A9E86/5F64E7E9/5FF1EA9B" Ref="R52"  Part="1"
 AR Path="/5F4A9E86/5F6DDF02/5FF1EA9B" Ref="R58"  Part="1"
-F 0 "R46" V 4400 3700 50  0000 C CNN
+F 0 "R58" V 4400 3700 50  0000 C CNN
 F 1 "10k" V 4500 3700 50  0000 C CNN
 F 2 "Resistor_SMD:R_0402_1005Metric" V 4430 3700 50  0001 C CNN
@@
 AR Path="/5F4A9E86/5F64E7E9/5FF1F393" Ref="R53"  Part="1"
 AR Path="/5F4A9E86/5F6DDF02/5FF1F393" Ref="R59"  Part="1"
-F 0 "R47" V 4600 3900 50  0000 C CNN
+F 0 "R59" V 4600 3900 50  0000 C CNN
 F 1 "10k" V 4500 3900 50  0000 C CNN
 F 2 "Resistor_SMD:R_0402_1005Metric" V 4430 3900 50  0001 C CNN
@@
 AR Path="/5F4A9E86/5F64E7E9/5FF1F59B" Ref="R54"  Part="1"
 AR Path="/5F4A9E86/5F6DDF02/5FF1F59B" Ref="R60"  Part="1"
-F 0 "R48" H 4730 3354 50  0000 R CNN
+F 0 "R60" H 4730 3354 50  0000 R CNN
 F 1 "10k" H 4730 3445 50  0000 R CNN
 F 2 "Resistor_SMD:R_0402_1005Metric" V 4730 3400 50  0001 C CNN
@@
 AR Path="/5F4A9E86/5F64E7E9/5FF1F8A9" Ref="R55"  Part="1"
 AR Path="/5F4A9E86/5F6DDF02/5FF1F8A9" Ref="R61"  Part="1"
-F 0 "R49" H 5080 3354 50  0000 R CNN
+F 0 "R61" H 5080 3354 50  0000 R CNN
 F 1 "10k" H 5080 3445 50  0000 R CNN
 F 2 "Resistor_SMD:R_0402_1005Metric" V 5080 3400 50  0001 C CNN
@@
 AR Path="/5F4A9E86/5F64E7E9/5FF1FD2A" Ref="R57"  Part="1"
 AR Path="/5F4A9E86/5F6DDF02/5FF1FD2A" Ref="R63"  Part="1"
-F 0 "R51" H 7070 3496 50  0000 L CNN
+F 0 "R63" H 7070 3496 50  0000 L CNN
 F 1 "10k" H 7070 3405 50  0000 L CNN
 F 2 "Resistor_SMD:R_0402_1005Metric" V 6930 3450 50  0001 C CNN
@@
 AR Path="/5F4A9E86/5F6DDF02/5F6A38A0" Ref="C17"  Part="1"
 AR Path="/5F4A9E86/5F60074F/5F6A38A0" Ref="C?"  Part="1"
-F 0 "C11" H 7115 3996 50  0000 L CNN
+F 0 "C17" H 7115 3996 50  0000 L CNN
 F 1 "0.1uF" H 7115 3905 50  0000 L CNN
 F 2 "Capacitor_SMD:C_0402_1005Metric" H 7038 3800 50  0001 C CNN
@@
 AR Path="/5F4A9E86/5F64E7E9/6079BFA7" Ref="W6"  Part="1"
 AR Path="/5F4A9E86/5F64E1A9/6079BFA7" Ref="W4"  Part="1"
-F 0 "W5" H 6200 5550 50  0000 L CNN
+F 0 "W7" H 6200 5550 50  0000 L CNN
 F 1 "Cable Assembly (5 Wire)" H 5400 5450 50  0000 L CNN
 F 2 "" H 6450 5500 50  0001 C CNN
@@
 AR Path="/5F4A9E86/5F64E7E9/5FF1FAB4" Ref="R56"  Part="1"
 AR Path="/5F4A9E86/5F6DDF02/5FF1FAB4" Ref="R62"  Part="1"
-F 0 "R50" V 6850 3700 50  0000 C CNN
+F 0 "R62" V 6850 3700 50  0000 C CNN
 F 1 "1k" V 6750 3700 50  0000 C CNN
 F 2 "Resistor_SMD:R_0402_1005Metric" V 6680 3700 50  0001 C CNN
@@
 AR Path="/5F4A9E86/5F64E1A9/606FF852" Ref="J10"  Part="1"
 AR Path="/5F4A9E86/5F6DDF02/606FF852" Ref="J13"  Part="1"
-F 0 "J11" H 6330 5292 50  0000 L CNN
+F 0 "J13" H 6330 5292 50  0000 L CNN
 F 1 "EncoderConnector" H 6330 5201 50  0000 L CNN
 F 2 "Connector_JST:JST_PH_S5B-PH-K_1x05_P2.00mm_Horizontal" H 6250 5250 50  0001 C CNN
 F 3 "~" H 6250 5250 50  0001 C CNN
-F 4 "455-1752-1-ND" H 6250 5250 50  0001 C CNN "Digikey"
+F 4 "455-1722-ND" H 6250 5250 50  0001 C CNN "Digikey"
 	1    6250 5250
 	1    0    0    1
