File: PCB/V2/Power.sch (KiCad schematic (older format))
At the start: 24 parts, among them J8 Barrel_Jack_Switch, Q1 FDN338P, Q2 MMBT3904, Q3 FDN338P, U7 DMP1005UFDF, U8 AP2114HA-3.3TRG1

Commit message: PCB Sent
Parts:
- C35, C36, C38: footprint Capacitor_SMD:C_1206_3216Metric -> Capacitor_SMD:C_0805_2012Metric; Digikey 1276-1055-1-ND -> 1276-1244-1-ND
- C37: Digikey 1276-6687-1-ND -> 1276-2909-1-ND
- D15: Digikey 160-1446-1-ND -> 160-1183-1-ND
- Q1, Q3: value FDN338P -> CPH3356-TL-W; Digikey FDN338PCT-ND -> CPH3356-TL-WOSCT-ND
- U8: Digikey AP2114HA-3.3TRG1 -> AP2114HA-3.3TRG1DICT-ND
Changed lines of the file:
@@
 F 2 "Package_TO_SOT_SMD:SOT-223-3_TabPin2" H 8000 1650 50  0001 C CNN
 F 3 "https://www.diodes.com/assets/Datasheets/AP2114.pdf" H 8000 1650 50  0001 C CNN
-F 4 "AP2114HA-3.3TRG1" H 8000 1650 50  0001 C CNN "Digikey"
+F 4 "AP2114HA-3.3TRG1DICT-ND" H 8000 1650 50  0001 C CNN "Digikey"
 F 5 "AP2114HA-3.3TRG1DICT-ND" H 8000 1650 50  0001 C CNN "MPN"
 F 6 "Diodes Inc." H 8000 1650 50  0001 C CNN "Manufacturer"
@@
 F 0 "C38" H 8965 1946 50  0000 L CNN
 F 1 "4.7uF" H 8965 1855 50  0000 L CNN
-F 2 "Capacitor_SMD:C_1206_3216Metric" H 8888 1750 50  0001 C CNN
+F 2 "Capacitor_SMD:C_0805_2012Metric" H 8888 1750 50  0001 C CNN
 F 3 "~" H 8850 1900 50  0001 C CNN
-F 4 "1276-1055-1-ND" H 8850 1900 50  0001 C CNN "Digikey"
+F 4 "1276-1244-1-ND" H 8850 1900 50  0001 C CNN "Digikey"
 F 5 "Samsung" H 8850 1900 50  0001 C CNN "Manufacturer"
 F 6 "CL31B475KAHNNNE" H 8850 1900 50  0001 C CNN "MPN"
@@
 F 0 "C35" H 5165 3446 50  0000 L CNN
 F 1 "4.7uF" H 5165 3355 50  0000 L CNN
-F 2 "Capacitor_SMD:C_1206_3216Metric" H 5088 3250 50  0001 C CNN
+F 2 "Capacitor_SMD:C_0805_2012Metric" H 5088 3250 50  0001 C CNN
 F 3 "~" H 5050 3400 50  0001 C CNN
-F 4 "1276-1055-1-ND" H 5050 3400 50  0001 C CNN "Digikey"
+F 4 "1276-1244-1-ND" H 5050 3400 50  0001 C CNN "Digikey"
 F 5 "Samsung" H 5050 3400 50  0001 C CNN "Manufacturer"
 F 6 "CL31B475KAHNNNE" H 5050 3400 50  0001 C CNN "MPN"
@@
 AR Path="/5F8CC9DA/5F8D3895" Ref="Q1"  Part="1"
 F 0 "Q1" V 3850 4800 50  0000 L CNN
-F 1 "FDN338P" V 3950 4600 50  0000 L CNN
+F 1 "CPH3356-TL-W" V 3950 4600 50  0000 L CNN
 F 2 "Package_TO_SOT_SMD:SOT-23" H 4200 5200 50  0001 C CNN
 F 3 "https://www.onsemi.com/pub/Collateral/FDN338P-D.pdf" H 4000 5100 50  0001 C CNN
-F 4 "FDN338PCT-ND" H 4000 5100 50  0001 C CNN "Digikey"
+F 4 "CPH3356-TL-WOSCT-ND" H 4000 5100 50  0001 C CNN "Digikey"
 	1    4000 5100
 	0    -1   -1   0
@@
 F 0 "C36" H 6915 1946 50  0000 L CNN
 F 1 "4.7uF" H 6915 1855 50  0000 L CNN
-F 2 "Capacitor_SMD:C_1206_3216Metric" H 6838 1750 50  0001 C CNN
+F 2 "Capacitor_SMD:C_0805_2012Metric" H 6838 1750 50  0001 C CNN
 F 3 "~" H 6800 1900 50  0001 C CNN
-F 4 "1276-1055-1-ND" H 6800 1900 50  0001 C CNN "Digikey"
+F 4 "1276-1244-1-ND" H 6800 1900 50  0001 C CNN "Digikey"
 F 5 "Samsung" H 6800 1900 50  0001 C CNN "Manufacturer"
 F 6 "CL31B475KAHNNNE" H 6800 1900 50  0001 C CNN "MPN"
@@
 AR Path="/5F8CC9DA/5F8D3900" Ref="Q3"  Part="1"
 F 0 "Q3" H 8450 4300 50  0000 L CNN
-F 1 "FDN338P" H 8400 4400 50  0000 L CNN
+F 1 "CPH3356-TL-W" H 8400 4400 50  0000 L CNN
 F 2 "Package_TO_SOT_SMD:SOT-23" H 8400 4500 50  0001 C CNN
 F 3 "https://www.onsemi.com/pub/Collateral/FDN338P-D.pdf" H 8200 4400 50  0001 C CNN
-F 4 "FDN338PCT-ND" H 8200 4400 50  0001 C CNN "Digikey"
+F 4 "CPH3356-TL-WOSCT-ND" H 8200 4400 50  0001 C CNN "Digikey"
 	1    8200 4400
 	1    0    0    1
@@
 F 2 "LED_SMD:LED_0603_1608Metric" H 4150 1850 50  0001 C CNN
 F 3 "~" H 4150 1850 50  0001 C CNN
-F 4 "160-1446-1-ND" H 4150 1850 50  0001 C CNN "Digikey"
+F 4 "160-1183-1-ND" H 4150 1850 50  0001 C CNN "Digikey"
 F 5 "LTST-C191KGKT" H 4150 1850 50  0001 C CNN "MPN"
 F 6 "Lite-On Inc." H 4150 1850 50  0001 C CNN "Manufacturer"
@@
 F 2 "Capacitor_SMD:C_0805_2012Metric" H 7250 1900 50  0001 C CNN
 F 3 "~" H 7250 1900 50  0001 C CNN
-F 4 "1276-6687-1-ND" H 7250 1900 50  0001 C CNN "Digikey"
+F 4 "1276-2909-1-ND" H 7250 1900 50  0001 C CNN "Digikey"
 F 5 "CL21A226KQCLRNC" H 7250 1900 50  0001 C CNN "MPN"
 F 6 "Samsung" H 7250 1900 50  0001 C CNN "Manufacturer"
