File: PCB/V2/QuadEncoder.sch (KiCad schematic (older format))
At the start: 35 parts, among them J1 SliderConnector, J2 SliderConnector, J9 SliderConnector, SW1 SW_Push_LED, SW2 SW_Push_LED, SW3 SW_Push_LED, SW4 SW_Push_LED, SW5 SW_Push_LED, SW6 SW_Push_LED, U2 MCP23017_SO

Commit message: PCB Sent
Parts:
- C5: footprint Capacitor_SMD:C_1206_3216Metric -> Capacitor_SMD:C_0805_2012Metric; Digikey 1276-1055-1-ND -> 1276-1244-1-ND
- J1, J2, J9: footprint Connector_JST:JST_EH_B3B-EH-A_1x03_P2.50mm_Vertical -> Connector_JST:JST_PH_S3B-PH-K_1x03_P2.00mm_Horizontal; Digikey 455-1721-ND -> 455-1720-ND
- U2: Digikey MCP23017T-E/SOCT-ND -> MCP23017-E/SO; MPN MCP23017T-E/SO -> MCP23017-E/SO
- W1, W2, W3: Digikey 1460-1291-ND -> 1528-4336-ND
Connections:
- net +3V3: now also J1.2 (Pin_2), J2.2 (Pin_2), J9.2 (Pin_2); no longer J1.1 (Pin_1), J2.1 (Pin_1), J9.1 (Pin_1)
- net GND: now also R3.2, R4.2, R5.2, R6.2, R7.2, R8.2; no longer SW1.3 (K), SW2.3 (K), SW3.3 (K), SW4.3 (K), SW5.3 (K), SW6.3 (K)
- net LED_Power: now also SW1.4 (A), SW2.4 (A), SW3.4 (A), SW4.4 (A), SW5.4 (A), SW6.4 (A); no longer R3.1, R4.1, R5.1, R6.1, R7.1, R8.1
- net SLD1: now also J1.1 (Pin_1); no longer J1.2 (Pin_2)
- net SLD2: now also J2.1 (Pin_1); no longer J2.2 (Pin_2)
- net SLD3: now also J9.1 (Pin_1); no longer J9.2 (Pin_2)
- new net: R3.1, SW1.3 (K)
- new net: R5.1, SW3.3 (K)
- new net: R7.1, SW5.3 (K)
- new net: R4.1, SW2.3 (K)
- new net: R6.1, SW4.3 (K)
- new net: R8.1, SW6.3 (K)
Other:
- note added: "B"
- note added: "R"
- note added: "W"
- moved on the sheet: J1, R3, R4, R5, R6, R7, R8
