File: PCB/V2/USB.sch (KiCad schematic (older format))
At the start: 50 parts, among them J3 USB_B, J4 USB_A, J5 USB_A, J6 USB_A, J7 USB_A, U3 CY7C65632-28LTXC, U4 24LC02, U5 MIC2027, Y2 12MHz

Commit message: PCB Sent
Parts:
- U4: Digikey 24LC02BT/SN -> 24LC02BT/SNCT-ND
Changed lines of the file:
@@
 F 2 "Package_SO:SOIC-8_3.9x4.9mm_P1.27mm" H 4300 8700 50  0001 C CNN
 F 3 "http://ww1.microchip.com/downloads/en/DeviceDoc/21709c.pdf" H 4300 8700 50  0001 C CNN
-F 4 "24LC02BT/SN" H 4300 8700 50  0001 C CNN "Digikey"
+F 4 "24LC02BT/SNCT-ND" H 4300 8700 50  0001 C CNN "Digikey"
 F 5 "24LC02BT/SNCT-ND" H 4300 8700 50  0001 C CNN "MPN"
 F 6 "Microchip" H 4300 8700 50  0001 C CNN "Manufacturer"
